File: z80/z80.sch (KiCad schematic (older format))
At the start: 94 parts, among them SW1 SW_Push, X8.000Mhz TFT680

Commit message: * Added Arduino Programmer code, Schematic changes
Parts:
- removed SW?: SW_SPST, symbol Switch:SW_SPST
- added SW? (x4): SW_SPST, symbol Switch:SW_SPST
- added SW? (x2): SW_DPDT_x2, symbol Switch:SW_DPDT_x2
- added U? (x2): 74AUC2G32, symbol 74xGxx:74AUC2G32
- A?: symbol MCU_Module:Arduino_Leonardo -> promicro:Sparkfun_Pro_Micro
Connections:
- net +5V: now also U?.10 (~SRCLR), U?.10 (~SRCLR), SW?.2 (B); no longer A?.5 (+5V)
- net A14: now also U?.1
- net A15: now also U?.2
- net GND: now also U?.13 (~OE), U?.13 (~OE), SW?.1 (A), SW?.2 (B), SW?.3 (C), U?.4 (GND), U?.4 (GND); no longer A?.6 (GND)
- net RD: now also SW?.1 (A); no longer ROM.22 (*OE), U?.6 (QG)
- net VCC: now also U?.8 (VCC), U?.8 (VCC)
- net WR: no longer ROM.27 (*WE), U?.5 (QF)
- net at U?.2: now also U?.2; no longer U?.2
- net at U?.7: now also SW?.3 (C); no longer ROM.20 (*CE)
- net at A?.9 (A0): now also SW?.1 (A)
- net at R?.1: now also SW?.2 (B)
- new net: A?.5 (+5V), SW?.1 (A)
- new net: A?.6 (GND), SW?.1 (A)
- new net: U?.2, U?.7
- new net: ROM.20 (*CE), SW?.2 (B)
- new net: U?.1, U?.7
- new net PRD: ROM.22 (*OE), SW?.2 (B), SW?.2 (B)
- new net PWR: A?.25 (D10), ROM.27 (*WE)
- no-connect marks 5 -> 26

Commit message: Added python programmer interface
Parts:
- added J0: Conn_02x14_Counter_Clockwise, symbol Connector_Generic:Conn_02x14_Counter_Clockwise
- added U0: SST39SF040, symbol Memory_Flash:SST39SF040
- added U1, U?: 74LS174, symbol 74xx:74LS174
- added U?: 4069, symbol z80-rescue:4069-4xxx
- gave numbers to parts that had none: 7
Connections:
- net +5V: now also U?.16 (VCC)
- net GND: now also U0.16 (GND), U?.8 (GND)
- net VCC: now also U0.32 (VCC)
- new net: U0.1 (A18), U1.10 (Q3)
- new net: U0.2 (A16), U1.5 (Q1)
- new net: U0.3 (A15), U1.2 (Q0)
- new net: U0.30 (A17), U1.7 (Q2)
- no-connect marks 26 -> 28
Changed lines of the file:
@@
 System Memory
 $Comp
-L 74xx:74LS174 U?
+L 74xx:74LS174 U0
 U 1 1 617C7373
 P 15250 7100
-F 0 "U?" H 15250 7981 50  0001 C CNN
+F 0 "U0" H 15000 7650 50  0000 C CNN
 F 1 "74LS174" H 15450 7650 50  0000 C CNN
 F 2 "" H 15250 7100 50  0001 C CNN
@@
 $EndComp
 $Comp
-L z80-rescue:4081-4xxx U?
+L z80-rescue:4081-4xxx U2
 U 5 1 617E86AE
 P 13800 6450
-F 0 "U?" V 13433 6450 50  0001 C CNN
+F 0 "U2" V 13650 6850 50  0000 C CNN
 F 1 "4081" V 13524 6450 50  0001 C CNN
 F 2 "" H 13800 6450 50  0001 C CNN
@@
 $EndComp
 $Comp
-L z80-rescue:4081-4xxx U?
+L z80-rescue:4081-4xxx U2
 U 4 1 617E2BC1
 P 13700 7900
-F 0 "U?" H 13700 8225 50  0001 C CNN
+F 0 "U2" H 13450 7900 50  0000 C CNN
 F 1 "4081" H 13700 8134 50  0001 C CNN
 F 2 "" H 13700 7900 50  0001 C CNN
@@
 $EndComp
 $Comp
-L z80-rescue:4081-4xxx U?
+L z80-rescue:4081-4xxx U2
 U 3 1 617E1936
 P 13700 7550
-F 0 "U?" H 13700 7875 50  0001 C CNN
+F 0 "U2" H 13450 7550 50  0000 C CNN
 F 1 "4081" H 13700 7784 50  0001 C CNN
 F 2 "" H 13700 7550 50  0001 C CNN
@@
 $EndComp
 $Comp
-L z80-rescue:4081-4xxx U?
+L z80-rescue:4081-4xxx U2
 U 2 1 617DFD9C
 P 13700 7200
-F 0 "U?" H 13700 7525 50  0001 C CNN
+F 0 "U2" H 13450 7200 50  0000 C CNN
 F 1 "4081" H 13700 7434 50  0001 C CNN
 F 2 "" H 13700 7200 50  0001 C CNN
@@
 $EndComp
 $Comp
-L z80-rescue:4081-4xxx U?
+L z80-rescue:4081-4xxx U2
 U 1 1 617D8F89
 P 13700 6850
-F 0 "U?" H 13700 7175 50  0001 C CNN
+F 0 "U2" H 13450 6850 50  0000 C CNN
 F 1 "4081" H 13700 7084 50  0001 C CNN
 F 2 "" H 13700 6850 50  0001 C CNN
@@
 $EndComp
 $Comp
-L z80-rescue:4081-4xxx U?
+L z80-rescue:4081-4xxx U3
 U 1 1 61830A0B
 P 13700 8250
-F 0 "U?" H 13700 8575 50  0001 C CNN
+F 0 "U3" H 13450 8250 50  0000 C CNN
 F 1 "4081" H 13700 8484 50  0001 C CNN
 F 2 "" H 13700 8250 50  0001 C CNN
@@
 $EndComp
 $Comp
-L z80-rescue:4081-4xxx U?
+L z80-rescue:4081-4xxx U3
 U 2 1 61832086
 P 13700 8600
-F 0 "U?" H 13700 8925 50  0001 C CNN
+F 0 "U3" H 13450 8600 50  0000 C CNN
 F 1 "4081" H 13700 8834 50  0001 C CNN
 F 2 "" H 13700 8600 50  0001 C CNN
@@
 $EndComp
 $Comp
-L z80-rescue:4081-4xxx U?
+L z80-rescue:4081-4xxx U3
 U 3 1 6183366C
 P 13700 8950
-F 0 "U?" H 13700 9275 50  0001 C CNN
+F 0 "U3" H 13450 8950 50  0000 C CNN
 F 1 "4081" H 13700 9184 50  0001 C CNN
 F 2 "" H 13700 8950 50  0001 C CNN
@@
 $EndComp
 $Comp
-L z80-rescue:4081-4xxx U?
+L z80-rescue:4081-4xxx U3
 U 4 1 61834DB5
 P 13700 9300
-F 0 "U?" H 13700 9625 50  0001 C CNN
+F 0 "U3" H 13450 9300 50  0000 C CNN
 F 1 "4081" H 13700 9534 50  0001 C CNN
 F 2 "" H 13700 9300 50  0001 C CNN
@@
 $EndComp
 $Comp
-L z80-rescue:4081-4xxx U?
+L z80-rescue:4081-4xxx U3
 U 5 1 6183680D
 P 13800 9700
-F 0 "U?" V 13433 9700 50  0001 C CNN
+F 0 "U3" V 13950 10100 50  0000 C CNN
 F 1 "4081" V 13524 9700 50  0001 C CNN
 F 2 "" H 13800 9700 50  0001 C CNN
@@
 $EndComp
 $Comp
-L 74xx:74LS174 U?
+L 74xx:74LS174 U1
 U 1 1 6187FAE0
 P 15250 8950
-F 0 "U?" H 15250 9831 50  0001 C CNN
+F 0 "U1" H 15000 9500 50  0000 C CNN
 F 1 "74LS174" H 15450 9500 50  0000 C CNN
 F 2 "" H 15250 8950 50  0001 C CNN
@@
 A0
 $Comp
-L 74xGxx:74AUC2G32 U?
+L 74xGxx:74AUC2G32 U5
 U 1 1 61B34189
 P 12250 9200
-F 0 "U?" H 12200 9500 50  0001 C CNN
+F 0 "U5" V 12150 9400 50  0001 C CNN
 F 1 "74AUC2G32" H 12225 9376 50  0001 C CNN
 F 2 "" H 12250 9200 50  0001 C CNN
@@
 $EndComp
 $Comp
-L z80-rescue:4069-4xxx U?
+L z80-rescue:4069-4xxx U4
 U 1 1 61B37C38
 P 12550 9450
-F 0 "U?" H 12550 9133 50  0001 C CNN
+F 0 "U4" H 12650 9550 50  0000 C CNN
 F 1 "4069" H 12550 9224 50  0001 C CNN
 F 2 "" H 12550 9450 50  0001 C CNN
@@
 IOReq
 $Comp
-L 74xx:74HC595 U?
+L 74xx:74HC595 U0
 U 1 1 61730099
 P 3400 8100
-F 0 "U?" H 3400 8881 50  0001 C CNN
+F 0 "U0" H 3150 8650 50  0000 C CNN
 F 1 "74HC595" H 3400 8790 50  0001 C CNN
 F 2 "" H 3400 8100 50  0001 C CNN
@@
 $EndComp
 $Comp
-L promicro:Sparkfun_Pro_Micro A?
+L promicro:Sparkfun_Pro_Micro A0
 U 1 1 6173E89B
 P 1250 8950
-F 0 "A?" H 1250 10131 50  0001 C CNN
+F 0 "A0" H 1050 7800 50  0000 C CNN
 F 1 "32U4 Arduino" H 850 7900 50  0000 C CNN
 F 2 "Module:Arduino_UNO_R3" H 1250 8950 50  0001 C CIN
@@
 RD
 $Comp
-L 74xx:74HC595 U?
+L 74xx:74HC595 U1
 U 1 1 617346A3
 P 3400 9950
-F 0 "U?" H 3400 10731 50  0001 C CNN
+F 0 "U1" H 3150 10500 50  0000 C CNN
 F 1 "74HC595" H 3400 10640 50  0001 C CNN
 F 2 "" H 3400 9950 50  0001 C CNN
@@
 	0    -1   -1   0
 $EndComp
+$Comp
+L 74xx:74LS174 U?
+U 1 1 619D0860
+P 9700 6800
+F 0 "U?" H 9700 7681 50  0001 C CNN
+F 1 "74LS174" H 9900 7350 50  0000 C CNN
+F 2 "" H 9700 6800 50  0001 C CNN
+F 3 "http://www.ti.com/lit/gpn/sn74LS174" H 9700 6800 50  0001 C CNN
+	1    9700 6800
+	1    0    0    -1
+$EndComp
+$Comp
+L z80-rescue:4069-4xxx U?
+U 1 1 619D223C
+P 10050 8100
+F 0 "U?" H 10050 7783 50  0001 C CNN
+F 1 "4069" H 10050 7874 50  0001 C CNN
+F 2 "" H 10050 8100 50  0001 C CNN
+F 3 "http://www.intersil.com/content/dam/Intersil/documents/cd40/cd4069ubms.pdf" H 10050 8100 50  0001 C CNN
+	1    10050 8100
+	1    0    0    -1
+$EndComp
+$Comp
+L power:+5V #PWR?
+U 1 1 619D27CF
+P 9700 6100
+F 0 "#PWR?" H 9700 5950 50  0001 C CNN
+F 1 "+5V" H 9600 6100 50  0000 C CNN
+F 2 "" H 9700 6100 50  0001 C CNN
+F 3 "" H 9700 6100 50  0001 C CNN
+	1    9700 6100
+	1    0    0    -1
+$EndComp
+$Comp
+L power:GND #PWR?
+U 1 1 619D2CF2
+P 9700 7600
+F 0 "#PWR?" H 9700 7350 50  0001 C CNN
+F 1 "GND" H 9800 7600 50  0000 C CNN
+F 2 "" H 9700 7600 50  0001 C CNN
+F 3 "" H 9700 7600 50  0001 C CNN
+	1    9700 7600
+	1    0    0    -1
+$EndComp
+$Comp
+L Memory_Flash:SST39SF040 U0
+U 1 1 619D51EE
+P 14400 2400
+F 0 "U0" H 14750 3700 50  0000 C CNN
+F 1 "SST39SF040" H 14100 3700 50  0000 C CNN
+F 2 "" H 14400 2700 50  0001 C CNN
+F 3 "http://ww1.microchip.com/downloads/en/DeviceDoc/25022B.pdf" H 14400 2700 50  0001 C CNN
+	1    14400 2400
+	1    0    0    -1
+$EndComp
+$Comp
+L 74xx:74LS174 U1
+U 1 1 619DA82A
+P 13000 3100
+F 0 "U1" H 12750 3650 50  0000 C CNN
+F 1 "74LS174" H 13200 3650 50  0000 C CNN
+F 2 "" H 13000 3100 50  0001 C CNN
+F 3 "http://www.ti.com/lit/gpn/sn74LS174" H 13000 3100 50  0001 C CNN
+	1    13000 3100
+	1    0    0    -1
+$EndComp
+Wire Wire Line
+	13500 2700 13800 2700
+Wire Wire Line
+	13800 2800 13500 2800
+Wire Wire Line
+	13500 2900 13800 2900
+Wire Wire Line
+	13800 3000 13500 3000
+NoConn ~ 13500 3100
+NoConn ~ 13500 3200
+$Comp
+L Connector_Generic:Conn_02x14_Counter_Clockwise J0
+U 1 1 61A00789
+P 14350 4150
+F 0 "J0" V 14400 4830 50  0000 L CNN
+F 1 "Conn_02x14_Counter_Clockwise" V 14445 4830 50  0001 L CNN
+F 2 "" H 14350 4150 50  0001 C CNN
+F 3 "~" H 14350 4150 50  0001 C CNN
+	1    14350 4150
+	0    1    1    0
+$EndComp
 $EndSCHEMATC

Commit message: schematic changes
Parts:
- removed J0: Conn_02x14_Counter_Clockwise, symbol Connector_Generic:Conn_02x14_Counter_Clockwise
- removed SW?: SW_SPST, symbol Switch:SW_SPST
- added J?: Conn_02x16_Counter_Clockwise, symbol Connector_Generic:Conn_02x16_Counter_Clockwise
- added R? (x4): 1K, symbol Device:R_Small
- added SW? (x2): SW_SPDT, symbol Switch:SW_SPDT
- added U?: 74LS174, symbol 74xx:74LS174
Connections:
- net +5V: now also SW?.1 (A), SW?.3 (C), U?.16 (VCC)
- net A15: now also J?.9 (Pin_9)
- net GND: now also U1.13 (D4), U1.14 (D5), U1.8 (GND), J?.16 (Pin_16), J?.17 (Pin_17), SW?.3 (C), U?.8 (GND)
- net PRD: now also SW?.2 (B)
- net RD: now also J?.14 (Pin_14)
- net VCC: now also ROM.27 (*WE), U1.16 (VCC), J?.10 (Pin_10), R?.2, SW?.2 (B)
- net WR: now also J?.15 (Pin_15)
- net at A0.9 (A0): now also SW?.1 (A)
- net at U0.1 (~Mr): now also R?.1
- net at U1.1 (~Mr): now also R?.1 (x2)
- net Reset: now reaches R?.1, SW?.2 (B)
- net Reset: now also R?.2, R?.2
- net at U0.31 (PGM): now also R?.1
- net PWR: no longer names the net of A0.25 (D10)
- net PWR: now also SW?.1 (A); no longer ROM.27 (*WE)
- new net IO: J?.12 (Pin_12)
- new net MEM: J?.13 (Pin_13)
- new net RST: J?.11 (Pin_11), R?.2
