File: z80/z80.kicad_sch (KiCad schematic)
At the start: 128 parts, among them J1 Conn_02x16_Counter_Clockwise, J2 Conn_02x16_Counter_Clockwise, SW1 SW_DPDT_x2, SW1 SW_Push, SW10 SW_SPDT, SW12 SW_DIP_x08, SW2 SW_DPDT_x2, SW2 SW_SP3T, SW27 SW_DPDT_x2, SW3 SW_SPDT, SW5 SW_DIP_x08, SW6 SW_SPST, SW7 SW_SPST, SW8 SW_DIP_x08, SW9 SW_DIP_x08, U1 74HC595, U10 74AUC2G32, U11 74AUC2G32, U12 74LS174, U13 74LS174, U14 74AUC2G32, U15 74AUC2G32, U16 74AUC2G32, U17 74AUC2G32, U18 74LS174, U19 4081, U2 74HC595, U20 4081, U21 SST39SF040, U22 74LS174, U23 74LS174, U3 74AUC2G32, U4 4069, U5 74AUC2G32, U6 74AUC2G32, U7 4069, U8 74AUC2G32, U9 4081, X8.000Mhz1 TFT680

Commit message: schematic and pcb changes
Parts:
- added R2: 1K, Resistor_SMD:R_0603_1608Metric_Pad0.98x0.95mm_HandSolder, symbol Device:R_Small
- added R3, R4, R5: 10K, Resistor_SMD:R_0603_1608Metric_Pad0.98x0.95mm_HandSolder, symbol Device:R_Small
- added U1: 4081, symbol z80-rescue:4081-4xxx
- added U4: (no value), symbol atf16v8bql:ATF16V8BQL-15PU
- C1, C6: footprint (none) -> Capacitor_SMD:C_0805_2012Metric_Pad1.18x1.45mm_HandSolder
- C2: renamed from C7; footprint (none) -> Capacitor_SMD:C_0805_2012Metric_Pad1.18x1.45mm_HandSolder
- C3: renamed from C4; footprint (none) -> Capacitor_SMD:C_0805_2012Metric_Pad1.18x1.45mm_HandSolder
- C4: renamed from C2; footprint (none) -> Capacitor_SMD:C_0805_2012Metric_Pad1.18x1.45mm_HandSolder
- C5: renamed from C3; footprint (none) -> Capacitor_SMD:C_0805_2012Metric_Pad1.18x1.45mm_HandSolder
- C7: renamed from C5; footprint (none) -> Capacitor_SMD:C_0805_2012Metric_Pad1.18x1.45mm_HandSolder
- D1, D2: value (none) -> LED; footprint (none) -> LED_SMD:LED_0603_1608Metric_Pad1.05x0.95mm_HandSolder
- D10, D11, D12, D13, D14, D15, D16, D17, D19, D20, D21, D22, D23, D24, D25, D26, D3, D4, D5, D6, D7, D8, D9: footprint (none) -> LED_SMD:LED_0603_1608Metric_Pad1.05x0.95mm_HandSolder
- D18: value (none) -> LED_Small; footprint (none) -> LED_SMD:LED_0603_1608Metric_Pad1.05x0.95mm_HandSolder
- R1: renamed from R4; footprint (none) -> Resistor_SMD:R_0603_1608Metric_Pad0.98x0.95mm_HandSolder
- R10: renamed from R5; value (none) -> 10K; footprint (none) -> Resistor_SMD:R_0603_1608Metric_Pad0.98x0.95mm_HandSolder
- R11: renamed from R7; footprint (none) -> Resistor_SMD:R_0603_1608Metric_Pad0.98x0.95mm_HandSolder
- R12, R13, R14, R15, R16, R17, R18, R19, R20, R21, R22, R23, R24, R25, R26, R27: renamed from R?; value (none) -> 1K; footprint (none) -> Resistor_SMD:R_0603_1608Metric_Pad0.98x0.95mm_HandSolder
- R28, R29, R30, R31, R32, R33, R34, R35: renamed from R?; footprint (none) -> Resistor_SMD:R_0603_1608Metric_Pad0.98x0.95mm_HandSolder
- R36: renamed from R8; footprint (none) -> Resistor_SMD:R_0603_1608Metric_Pad0.98x0.95mm_HandSolder
- R37: renamed from R9; value (none) -> 10K; footprint (none) -> Resistor_SMD:R_0603_1608Metric_Pad0.98x0.95mm_HandSolder
- R38: renamed from R10; value (none) -> 10K; footprint (none) -> Resistor_SMD:R_0603_1608Metric_Pad0.98x0.95mm_HandSolder
- R39: renamed from R11; footprint (none) -> Resistor_SMD:R_0603_1608Metric_Pad0.98x0.95mm_HandSolder
- R40: renamed from R12; value (none) -> 1K; footprint (none) -> Resistor_SMD:R_0603_1608Metric_Pad0.98x0.95mm_HandSolder
- R41: renamed from R13; footprint (none) -> Resistor_SMD:R_0603_1608Metric_Pad0.98x0.95mm_HandSolder
- R42: renamed from R14; footprint (none) -> Resistor_SMD:R_0603_1608Metric_Pad0.98x0.95mm_HandSolder
- R43: renamed from R15; footprint (none) -> Resistor_SMD:R_0603_1608Metric_Pad0.98x0.95mm_HandSolder
- R44: renamed from R16; footprint (none) -> Resistor_SMD:R_0603_1608Metric_Pad0.98x0.95mm_HandSolder
- R45: renamed from R17; footprint (none) -> Resistor_SMD:R_0603_1608Metric_Pad0.98x0.95mm_HandSolder
- R46: renamed from R18; footprint (none) -> Resistor_SMD:R_0603_1608Metric_Pad0.98x0.95mm_HandSolder
- R47: renamed from R19; footprint (none) -> Resistor_SMD:R_0603_1608Metric_Pad0.98x0.95mm_HandSolder
- R48: renamed from R20; footprint (none) -> Resistor_SMD:R_0603_1608Metric_Pad0.98x0.95mm_HandSolder
- R49: renamed from R21; footprint (none) -> Resistor_SMD:R_0603_1608Metric_Pad0.98x0.95mm_HandSolder
- R50: renamed from R22; footprint (none) -> Resistor_SMD:R_0603_1608Metric_Pad0.98x0.95mm_HandSolder
- R51: renamed from R23; footprint (none) -> Resistor_SMD:R_0603_1608Metric_Pad0.98x0.95mm_HandSolder
- R6: renamed from R1; value (none) -> 1K
- R7: renamed from R3; footprint (none) -> Resistor_SMD:R_0603_1608Metric_Pad0.98x0.95mm_HandSolder
- R8: renamed from R6; footprint (none) -> Resistor_SMD:R_0603_1608Metric_Pad0.98x0.95mm_HandSolder
- R9: renamed from R2; value (none) -> 10K; footprint (none) -> Resistor_SMD:R_0603_1608Metric_Pad0.98x0.95mm_HandSolder
- RV1: value (none) -> 1M
- SW15: renamed from SW26; value (none) -> SW_DPDT_x2
- gave numbers to parts that had none: 2
- renumbered SW9 to SW10, SW10 to SW11, SW27 to SW16, SW1 to SW4, SW2 to SW8, SW8 to SW9, U8 to U10, U9 to U11, U10 to U12, U11 to U13, U12 to U14, U13 to U15, U14 to U16, U15 to U17, U16 to U18, U17 to U19, U1 to U2, U18 to U20, U19 to U21, U20 to U22, U21 to U23, U22 to U24, U23 to U25, U2 to U3, U3 to U5, U4 to U6, U5 to U7, U6 to U8, U7 to U9
Connections:
- net +5V: now also R2.1, U1.14 (VDD), U4.20 (VCC); no longer CLK1.5 (Q), R9.2, SW1.1 (A), SW8.2
- net Clock: now also U1.10, U1.3, U1.4; no longer SW8.3
- net FstClk: now also U1.1; no longer SW8.4
- net GND: now also R3.1, R4.1, R5.1, U1.7 (VSS), U4.10 (GND)
- net ManClk: now also U1.8; no longer SW8.1
- net Reset: no longer J1.11 (Pin_11), J2.11 (Pin_11), R11.1, R40.2, SW15.2 (B)
- new net: R3.2, SW8.1, U1.2
- new net: R5.2, SW8.4, U1.9
- new net: R2.2, SW8.3
- new net: R4.2, SW8.2, U1.6
- new net AdjClk: CLK1.5 (Q), R9.2, SW1.1 (A), U1.5
- new net RST: J1.11 (Pin_11), J2.11 (Pin_11), R11.1, R40.2, SW15.2 (B)
Other:
- moved on the sheet: SW15A, SW8

Commit message: cleaned up files, added script to launch programming tool
Parts:
- added J1: Screw_Terminal_01x02, symbol Connector:Screw_Terminal_01x02
- added U4, U5, U?: 74HC241, symbol 74xx:74HC244
- added U?: SN74HC138N, N16, symbol 74hc138:SN74HC138N
- U1: footprint (none) -> Package_SO:SO-14_3.9x8.65mm_P1.27mm
- U15: renamed from U4; value (none) -> ATF16V8BQL-15PU
- renumbered J1 to J2, J2 to J3, SW15 to SW13, SW13 to SW14, SW14 to SW15, U9 to U11, U11 to U14, U14 to U16, U15 to U17, U16 to U18, U17 to U19, U18 to U20, U19 to U21, U20 to U22, U21 to U23, U22 to U24, U23 to U25, U24 to U26, U25 to U27, U5 to U6, U6 to U7, U7 to U8, U8 to U9
Connections:
- net +5V: now also J1.1 (Pin_1); no longer U15.20 (VCC)
- net A0: now also J3.18 (Pin_18), U25.12 (A0), U4.18 (1Y0)
- net A1: now also J3.19 (Pin_19), U25.11 (A1), U4.16 (1Y1)
- net A10: now also J3.28 (Pin_28), U25.23 (A10), U5.14 (1Y2)
- net A11: now also J3.29 (Pin_29), U25.25 (A11), U5.12 (1Y3)
- net A12: now also J3.30 (Pin_30), U25.4 (A12), U5.3 (2Y0)
- net A13: now also J3.31 (Pin_31), U25.28 (A13)
- net A14: now also J3.32 (Pin_32), U25.29 (A14)
- net A2: now also J3.20 (Pin_20), U25.10 (A2), U4.14 (1Y2)
- net A3: now also J3.21 (Pin_21), U25.9 (A3), U4.12 (1Y3)
- net A4: now also J3.22 (Pin_22), U25.8 (A4), U4.3 (2Y0)
- net A5: now also J3.23 (Pin_23), U25.7 (A5), U4.5 (2Y1)
- net A6: now also J3.24 (Pin_24), U25.6 (A6), U4.7 (2Y2)
- net A7: now also J3.25 (Pin_25), U25.5 (A7), U4.9 (2Y3)
- net A8: now also J3.26 (Pin_26), U25.27 (A8), U5.18 (1Y0)
- net A9: now also J3.27 (Pin_27), U25.26 (A9), U5.16 (1Y1)
- net D0: now also J3.8 (Pin_8), U25.13 (D0)
- net D1: now also J3.7 (Pin_7), U25.14 (D1)
- net D2: now also J3.6 (Pin_6), U25.15 (D2)
- net D3: now also J3.5 (Pin_5), U25.17 (D3)
- net D4: now also J3.4 (Pin_4), U25.18 (D4)
- net D5: now also J3.3 (Pin_3), U25.19 (D5)
- net D6: now also J3.2 (Pin_2), U25.20 (D6)
- net D7: now also J3.1 (Pin_1), U25.21 (D7)
- net GND: now also J1.2 (Pin_2); no longer J3.16 (Pin_16), J3.17 (Pin_17), U15.10 (GND), U22.13 (D4), U22.14 (D5), U22.8 (GND), U25.16 (GND)
- net PA10: no longer ROM1.21 (A10)
- net PA11: no longer ROM1.23 (A11)
- net PA8: no longer ROM1.25 (A8)
- net PA9: no longer ROM1.24 (A9)
- net PD3: no longer ROM1.15 (I/O3)
- net PD4: no longer ROM1.16 (I/O4)
- net PD5: no longer ROM1.17 (I/O5)
- net PD6: no longer ROM1.18 (I/O6)
- net PD7: no longer ROM1.19 (I/O7)
- net PRD: no longer ROM1.22 (*OE)
- net VCC: no longer J3.10 (Pin_10), R41.2, ROM1.27 (*WE), SW11.2 (B), U22.16 (VCC), U25.32 (VCC)
- net HALT: now reaches CPU1.18 (~{HALT})
- net WAIT: now reaches CPU1.24 (~{WAIT})
- net M1: now reaches CPU1.27 (~{M1})
- net RFSH: now reaches CPU1.28 (~{RFSH})
- net at RAM1.20 (~{CS}): no longer U6.7
- net at U2.1 (QB): now also U4.4 (1A1); no longer SW14.2
- net at U2.15 (QA): now also U4.2 (1A0); no longer SW14.1
- net at U2.2 (QC): now also U4.6 (1A2); no longer SW14.3
- net at U2.3 (QD): now also U4.8 (1A3); no longer SW14.4
- net at U2.4 (QE): now also U4.17 (2A0); no longer SW14.5
- net at U2.5 (QF): now also U4.15 (2A1); no longer SW14.6
- net at U2.6 (QG): now also U4.13 (2A2); no longer SW14.7
- net at U2.7 (QH): now also U4.11 (2A3); no longer SW14.8
- net at U3.1 (QB): now also U5.4 (1A1); no longer SW15.2
- net at U3.15 (QA): now also U5.2 (1A0); no longer SW15.1
- net at U3.2 (QC): now also U5.6 (1A2); no longer SW15.3
- net at U3.3 (QD): now also U5.8 (1A3); no longer SW15.4
- net at U3.4 (QE): now also U5.17 (2A0); no longer SW15.5
- net at ROM1.20 (~{CE}): no longer SW16.2 (B)
- new net: J3.16 (Pin_16), J3.17 (Pin_17), U22.13 (D4), U22.14 (D5), U22.8 (GND), U25.16 (GND)
- new net PWR: J3.10 (Pin_10), R41.2, SW11.2 (B), U22.16 (VCC), U25.32 (VCC)
Other:
- moved on the sheet: SW14, SW15, SW8, U1A, U1B, U1C, U1E
