File: z80/z80.kicad_sch (KiCad schematic)
At the start: 115 parts, among them J1 Screw_Terminal_01x02, J2 Conn_02x16_Counter_Clockwise, SW11 SW_SPDT, SW13 SW_DPDT_x2, SW3 SW_SPDT, SW4 SW_Push, SW7 SW_SPST, SW8 SW_SP3T, U1 4081, U11 4069, U14 4081, U15 ATF16V8BQL-15PU, U16 74LS174, U17 74LS174, U18 74AUC2G32, U19 74AUC2G32, U2 74HC595, U20 74AUC2G32, U21 74AUC2G32, U23 4081, U24 4081, U26 74LS174, U27 74LS174, U3 74HC595, X8.000Mhz1 TFT680

Commit message: aaaaaa
Connections:
- net RAM1-CS: now also U?.13 (Y2); no longer U?.14 (Y1)
- net ROM1-CS: now also U?.14 (Y1)
Changed lines of the file:
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@@
     (company "T. van de Weg")
   )
+  (bus_alias "Data" (members ))
   (bus_alias "Address" (members ))
-  (bus_alias "Data" (members ))
+  (junction (at 174.625 166.37) (diameter 0) (color 0 0 0 0)
+  )
   (junction (at 237.49 203.2) (diameter 0) (color 0 0 0 0)
   )
@@
     (stroke (width 0) (type default) (color 0 0 0 0))
   )
+  (wire (pts (xy 174.625 163.83) (xy 174.625 166.37))
+    (stroke (width 0) (type default) (color 0 0 0 0))
+  )
   (bus (pts (xy 142.24 97.155) (xy 142.24 99.695))
     (stroke (width 0) (type default) (color 0 0 0 0))
@@
     (stroke (width 0) (type default) (color 0 0 0 0))
   )
-  (wire (pts (xy 174.625 163.83) (xy 184.15 163.83))
+  (wire (pts (xy 174.625 161.29) (xy 184.15 161.29))
     (stroke (width 0) (type default) (color 0 0 0 0))
   )
@@
     (effects (font (size 1.27 1.27)) (justify left bottom))
   )
-  (label "RAM1-CS" (at 184.15 163.83 180)
-    (effects (font (size 1.27 1.27)) (justify right bottom))
-  )
+  (label "RAM1-CS" (at 184.15 161.29 180)
+    (effects (font (size 1.27 1.27)) (justify right bottom))
+  )

Commit message: schematic changes
Parts:
- removed R36, R39, R49, R51: 1K, Resistor_SMD:R_0603_1608Metric_Pad0.98x0.95mm_HandSolder, symbol Device:R_Small
- removed R37, R38, R42, R43, R44, R45, R46, R47, R48, R50: 10K, Resistor_SMD:R_0603_1608Metric_Pad0.98x0.95mm_HandSolder, symbol Device:R_Small
- removed U11: 4069, symbol z80-rescue:4069-4xxx
- removed U14, U23, U24: 4081, symbol z80-rescue:4081-4xxx
- removed U15: ATF16V8BQL-15PU, symbol atf16v8bql:ATF16V8BQL-15PU
- removed U16, U17, U26, U27: 74LS174, Package_SO:SO-16_5.3x10.2mm_P1.27mm, symbol 74xx:74LS174
- removed U18, U19, U20, U21: 74AUC2G32, symbol 74xGxx:74AUC2G32
- removed U?: 74HC241, symbol 74xx:74HC244
- added D17, D18, D19, D20: LED_Small, LED_SMD:LED_0603_1608Metric_Pad1.05x0.95mm_HandSolder, symbol Device:LED_Small
- added U5: SN74HC138N, N16, symbol 74hc138:SN74HC138N
- added U6: 4069, symbol 4xxx:4069
- added U7: 82C55A, Package_DIP:DIP-40_W15.24mm, symbol Interface:82C55A
- gave numbers to parts that had none: 1
- renumbered D17 to D21, D18 to D22, D19 to D23, D20 to D24, D21 to D25, D22 to D26, D23 to D27, D24 to D28, D25 to D29, D26 to D30, R5 to R10, R3 to R2, R6 to R3, R7 to R4, R4 to R5, R2 to R6, R8 to R7, R9 to R8, R10 to R9, SW3 to SW1, SW4 to SW2, SW7 to SW3, SW11 to SW4, SW8 to SW5, SW13 to SW6
Connections:
- net +5V: now also U5.16 (VCC), U6.14 (VDD), U7.26 (VCC)
- net A0: now also U7.9 (A0)
- net A1: now also U7.8 (A1)
- net A5: now also U5.1 (A)
- net A6: now also U5.2 (B)
- net A7: now also U5.3 (C)
- net D0: now also U7.34 (D0)
- net D1: now also U7.33 (D1)
- net D2: now also U7.32 (D2)
- net D3: now also U7.31 (D3)
- net D4: now also U7.30 (D4)
- net D5: now also U7.29 (D5)
- net D6: now also U7.28 (D6)
- net D7: now also U7.27 (D7)
- net GND: now also U4.5 (~{G2B}), U5.5 (~{G2B}), U5.8 (GND), U6.7 (VSS), U7.7 (GND)
- net IORQ: now also U4.6 (G1), U5.4 (~{G2A})
- net MREQ: now also U4.4 (~{G2A}), U5.6 (G1)
- net RAM1-CS: now also D17.1 (K), D18.1 (K); no longer U4.13 (Y2)
- net RD: now also U7.5 (~{RD})
- net ROM1-CS: now also D19.1 (K), D20.1 (K); no longer U4.14 (Y1), U4.15 (Y0)
- net RST: now also U6.1
- net WR: now also U7.36 (~{WR})
- net BUSACK: now reaches CPU1.23 (~{BUSACK})
- net BUSRQ: now reaches CPU1.25 (~{BUSRQ})
- net at U4.12 (Y3): now also D17.2 (A)
- new net: U6.2, U7.35 (RESET)
- new net: D19.2 (A), U4.14 (Y1)
- new net: D18.2 (A), U4.13 (Y2)
- new net: D20.2 (A), U4.15 (Y0)
- new net IO1-CS: U5.15 (Y0), U7.6 (~{CS})
- no-connect marks 45 -> 31
Other:
- note added: "I/O Chip Select"
- note added: "Memory Chip Select"
- note removed: "8-bit Output Register"
- note removed: "Chip Select"
- moved on the sheet: J1

Commit message: OS asm, repo cleanup
Parts:
- removed SW1, SW4: SW_SPDT, symbol Switch:SW_SPDT
- removed SW3: SW_SPST, symbol Switch:SW_SPST
- added D1, D2, D3: LED_Small, LED_SMD:LED_0603_1608Metric_Pad1.05x0.95mm_HandSolder, symbol Device:LED_Small
- added R? (x2): 10K, Resistor_SMD:R_0603_1608Metric_Pad0.98x0.95mm_HandSolder, symbol Device:R_Small
- U1: symbol z80-rescue:4081-4xxx -> 4xxx:4081
- renumbered D7 to D10, D8 to D11, D9 to D12, D10 to D13, D11 to D14, D12 to D15, D13 to D16, D14 to D17, D15 to D18, D16 to D19, D17 to D20, D18 to D21, D19 to D22, D20 to D23, D21 to D24, D22 to D25, D23 to D26, D24 to D27, D25 to D28, D26 to D29, D27 to D30, D28 to D31, D29 to D32, D30 to D33, D1 to D4, D2 to D5, D3 to D6, D4 to D7, D5 to D8, D6 to D9
Connections:
- net +5V: now also A1.5 (+5V)
- net Clock: now also D1.1 (K), D2.1 (K), D3.1 (K); no longer U1.10, U1.3, U1.4
- net D0: now also A1.17 (D2/SDA)
- net D1: now also A1.18 (D3/SCL)
- net D2: now also A1.19 (D4)
- net D3: now also A1.20 (D5)
- net D4: now also A1.21 (D6)
- net D5: now also A1.22 (D7)
- net D6: now also A1.23 (D8)
- net D7: now also A1.24 (D9)
- net GND: now also A1.6 (GND), R?.1, R?.1; no longer U2.13 (~{OE}), U3.13 (~{OE})
- net RAM1-CS: now also R?.2
- net RD: now also A1.9 (A0)
- net ROM1-CS: now also R?.2
- net RST: now also A1.25 (D10), U2.13 (~{OE}), U3.13 (~{OE})
- net WR: now also A1.10 (A1)
- new net: D1.2 (A), U1.3
- new net: D3.2 (A), U1.10
- new net: D2.2 (A), U1.4
- no-connect marks 31 -> 30
Other:
- moved on the sheet: SW5, U1A, U1B, U1C

Commit message: Schematic changes, test script
Parts:
- removed D20: LED_Small, LED_SMD:LED_0603_1608Metric_Pad1.05x0.95mm_HandSolder, symbol Device:LED_Small
- removed R12, R13, R15, R17, R19, R20, R21, R22, R23, R24, R25, R26, R27, R28, R29, R30, R31, R32, R33, R34, R35: 1K, Resistor_SMD:R_0603_1608Metric_Pad0.98x0.95mm_HandSolder, symbol Device:R_Small
- removed R? (x2): 10K, Resistor_SMD:R_0603_1608Metric_Pad0.98x0.95mm_HandSolder, symbol Device:R_Small
- removed SW6: SW_DPDT_x2, symbol Switch:SW_DPDT_x2
- added C8: 1uF, Capacitor_SMD:C_0603_1608Metric, symbol Device:C_Small
- added D1, D3, D7: D, symbol Device:D_Small
- added D24, D25, D26, D27, D28, D29, D30, D31, D32, D33: LED_Red, LED_SMD:LED_0603_1608Metric, symbol Device:LED_Small
- added J3: PinHeader_Female16x02, Card_Connector:FX2740S08SV, symbol Connector_Generic:Conn_02x20_Top_Bottom
- added J4, J5, J6, J7, J8, J9: PinHeader_Female04x02, Connector_PinSocket_2.54mm:PinSocket_2x04_P2.54mm_Vertical, symbol Connector_Generic:Conn_02x04_Top_Bottom
- added R10, R3: 1K, Resistor_SMD:R_0603_1608Metric, symbol Device:R_Small
- added R4: 10K, Resistor_SMD:R_0603_1608Metric, symbol Device:R_Small
- added RN1, RN2, RN3, RN4, RN5, RN6, RN7: EXB-D10C102J, r_network:EXB-D10C103J, symbol Device:R_Network08
- added SW3: SW_Push, Button_Switch_SMD:SW_SPST_B3S-1000, symbol Switch:SW_Push
- added unit 4 of U1
- added U10: 82C55A, Package_DIP:DIP-40_W15.24mm, symbol Interface:82C55A
- added unit 5 of U6
- added unit 6 of U6
- added unit 3 of U6
- added unit 2 of U6
- added unit 4 of U6
- added U8: 4081, Package_SO:SO-14_3.9x8.65mm_P1.27mm, symbol 4xxx:4081
- A1: footprint Package_DIP:DIP-24_W15.24mm_Socket -> (none)
- C1: footprint Capacitor_SMD:C_0805_2012Metric_Pad1.18x1.45mm_HandSolder -> Capacitor_SMD:C_0603_1608Metric; symbol Device:CP_Small -> Device:C_Small
- C2, C3, C4, C5, C6, C7: footprint Capacitor_SMD:C_0805_2012Metric_Pad1.18x1.45mm_HandSolder -> Capacitor_SMD:C_0603_1608Metric
- CLK1: footprint Package_DIP:DIP-14_W7.62mm_Socket -> Package_SO:SOIC-14_3.9x8.7mm_P1.27mm
- CPU1: value Z84C0010PEG -> Z84C0010AEG; footprint Package_DIP:DIP-40_W15.24mm_Socket -> Package_QFP:LQFP-44_10x10mm_P0.8mm
- D13: renamed from D26; value LED_Small -> LED_Yellow; footprint LED_SMD:LED_0603_1608Metric_Pad1.05x0.95mm_HandSolder -> LED_SMD:LED_0603_1608Metric
- D14: renamed from D27; value LED_Small -> LED_Yellow; footprint LED_SMD:LED_0603_1608Metric_Pad1.05x0.95mm_HandSolder -> LED_SMD:LED_0603_1608Metric
- D15: renamed from D28; value LED_Small -> LED_Yellow; footprint LED_SMD:LED_0603_1608Metric_Pad1.05x0.95mm_HandSolder -> LED_SMD:LED_0603_1608Metric
- D16: renamed from D29; value LED_Small -> LED_Yellow; footprint LED_SMD:LED_0603_1608Metric_Pad1.05x0.95mm_HandSolder -> LED_SMD:LED_0603_1608Metric
- D17: renamed from D30; value LED_Small -> LED_Yellow; footprint LED_SMD:LED_0603_1608Metric_Pad1.05x0.95mm_HandSolder -> LED_SMD:LED_0603_1608Metric
- D18: renamed from D31; value LED_Small -> LED_Yellow; footprint LED_SMD:LED_0603_1608Metric_Pad1.05x0.95mm_HandSolder -> LED_SMD:LED_0603_1608Metric
- D19: renamed from D32; value LED_Small -> LED_Yellow; footprint LED_SMD:LED_0603_1608Metric_Pad1.05x0.95mm_HandSolder -> LED_SMD:LED_0603_1608Metric
- D2: renamed from D1; value LED_Small -> LED_Blue; footprint LED_SMD:LED_0603_1608Metric_Pad1.05x0.95mm_HandSolder -> LED_SMD:LED_0603_1608Metric
- D20: renamed from D33; value LED_Small -> LED_Yellow; footprint LED_SMD:LED_0603_1608Metric_Pad1.05x0.95mm_HandSolder -> LED_SMD:LED_0603_1608Metric
- D21, D22, D23: value LED_Small -> LED_Red; footprint LED_SMD:LED_0603_1608Metric_Pad1.05x0.95mm_HandSolder -> LED_SMD:LED_0603_1608Metric
- D34: renamed from D6; value LED_Small -> LED_Yellow; footprint LED_SMD:LED_0603_1608Metric_Pad1.05x0.95mm_HandSolder -> LED_SMD:LED_0603_1608Metric
- D35: renamed from D7; value LED_Small -> LED_Yellow; footprint LED_SMD:LED_0603_1608Metric_Pad1.05x0.95mm_HandSolder -> LED_SMD:LED_0603_1608Metric
- D36: renamed from D8; value LED_Small -> LED_Yellow; footprint LED_SMD:LED_0603_1608Metric_Pad1.05x0.95mm_HandSolder -> LED_SMD:LED_0603_1608Metric
- D37: renamed from D9; value LED_Small -> LED_Yellow; footprint LED_SMD:LED_0603_1608Metric_Pad1.05x0.95mm_HandSolder -> LED_SMD:LED_0603_1608Metric
- D38: renamed from D10; value LED_Small -> LED_Yellow; footprint LED_SMD:LED_0603_1608Metric_Pad1.05x0.95mm_HandSolder -> LED_SMD:LED_0603_1608Metric
- D39: renamed from D11; value LED_Small -> LED_Yellow; footprint LED_SMD:LED_0603_1608Metric_Pad1.05x0.95mm_HandSolder -> LED_SMD:LED_0603_1608Metric
- D4: renamed from D2; value LED_Small -> LED_Blue; footprint LED_SMD:LED_0603_1608Metric_Pad1.05x0.95mm_HandSolder -> LED_SMD:LED_0603_1608Metric
- D40: renamed from D12; value LED_Small -> LED_Yellow; footprint LED_SMD:LED_0603_1608Metric_Pad1.05x0.95mm_HandSolder -> LED_SMD:LED_0603_1608Metric
- D41: renamed from D13; value LED_Small -> LED_Yellow; footprint LED_SMD:LED_0603_1608Metric_Pad1.05x0.95mm_HandSolder -> LED_SMD:LED_0603_1608Metric
- D42: renamed from D14; value LED_Small -> LED_Yellow; footprint LED_SMD:LED_0603_1608Metric_Pad1.05x0.95mm_HandSolder -> LED_SMD:LED_0603_1608Metric
- D43: renamed from D15; value LED_Small -> LED_Yellow; footprint LED_SMD:LED_0603_1608Metric_Pad1.05x0.95mm_HandSolder -> LED_SMD:LED_0603_1608Metric
- D44: renamed from D16; value LED_Small -> LED_Yellow; footprint LED_SMD:LED_0603_1608Metric_Pad1.05x0.95mm_HandSolder -> LED_SMD:LED_0603_1608Metric
- D45: renamed from D17; value LED_Small -> LED_Yellow; footprint LED_SMD:LED_0603_1608Metric_Pad1.05x0.95mm_HandSolder -> LED_SMD:LED_0603_1608Metric
- D46: renamed from D18; value LED_Small -> LED_Yellow; footprint LED_SMD:LED_0603_1608Metric_Pad1.05x0.95mm_HandSolder -> LED_SMD:LED_0603_1608Metric
- D47: renamed from D19; value LED_Small -> LED_Yellow; footprint LED_SMD:LED_0603_1608Metric_Pad1.05x0.95mm_HandSolder -> LED_SMD:LED_0603_1608Metric
- D48: renamed from D24; value LED_Small -> LED_Yellow; footprint LED_SMD:LED_0603_1608Metric_Pad1.05x0.95mm_HandSolder -> LED_SMD:LED_0603_1608Metric
- D49: renamed from D25; value LED_Small -> LED_Yellow; footprint LED_SMD:LED_0603_1608Metric_Pad1.05x0.95mm_HandSolder -> LED_SMD:LED_0603_1608Metric
- D5: renamed from D4; value LED -> LED_Blue; footprint LED_SMD:LED_0603_1608Metric_Pad1.05x0.95mm_HandSolder -> LED_SMD:LED_0603_1608Metric
- D6: renamed from D5; value LED -> LED_Blue; footprint LED_SMD:LED_0603_1608Metric_Pad1.05x0.95mm_HandSolder -> LED_SMD:LED_0603_1608Metric
- D8: renamed from D3; value LED_Small -> LED_Blue; footprint LED_SMD:LED_0603_1608Metric_Pad1.05x0.95mm_HandSolder -> LED_SMD:LED_0603_1608Metric
- J1: value Screw_Terminal_01x02 -> PinHeader_Female01x02; footprint (none) -> Connector_PinHeader_2.54mm:PinHeader_1x02_P2.54mm_Vertical
- J2: value Conn_02x16_Counter_Clockwise -> PinHeader_Female16x02; footprint Connector_PinSocket_2.54mm:PinSocket_2x16_P2.54mm_Vertical -> Card_Connector:FX2740S08SV; symbol Connector_Generic:Conn_02x16_Counter_Clockwise -> Connector_Generic:Conn_02x20_Top_Bottom
- R1, R14, R2: footprint Resistor_SMD:R_0603_1608Metric_Pad0.98x0.95mm_HandSolder -> Resistor_SMD:R_0603_1608Metric
- R11: renamed from R8; footprint Resistor_SMD:R_0603_1608Metric_Pad0.98x0.95mm_HandSolder -> Resistor_SMD:R_0603_1608Metric
- R12: renamed from R9; footprint Resistor_SMD:R_0603_1608Metric_Pad0.98x0.95mm_HandSolder -> Resistor_SMD:R_0603_1608Metric
- R13: renamed from R10; footprint Resistor_SMD:R_0603_1608Metric_Pad0.98x0.95mm_HandSolder -> Resistor_SMD:R_0603_1608Metric
- R15: renamed from R11; footprint Resistor_SMD:R_0603_1608Metric_Pad0.98x0.95mm_HandSolder -> Resistor_SMD:R_0603_1608Metric
- R16, R18: value 1K -> 10K; footprint Resistor_SMD:R_0603_1608Metric_Pad0.98x0.95mm_HandSolder -> Resistor_SMD:R_0603_1608Metric
- R6: renamed from R4; footprint Resistor_SMD:R_0603_1608Metric_Pad0.98x0.95mm_HandSolder -> Resistor_SMD:R_0603_1608Metric
- R7: renamed from R5; footprint Resistor_SMD:R_0603_1608Metric_Pad0.98x0.95mm_HandSolder -> Resistor_SMD:R_0603_1608Metric
- R8: renamed from R6; footprint Resistor_SMD:R_0603_1608Metric_Pad0.98x0.95mm_HandSolder -> Resistor_SMD:R_0603_1608Metric
- R9: renamed from R7; footprint Resistor_SMD:R_0603_1608Metric_Pad0.98x0.95mm_HandSolder -> Resistor_SMD:R_0603_1608Metric
- ROM1: footprint Package_DIP:DIP-28_W15.24mm_Socket -> Package_SO:SOIC-28W_7.5x17.9mm_P1.27mm; symbol PEEPROM:AT28C64B-15SU -> Atmel_EEPROM:AT28C64B
- RV1: footprint (none) -> Potentiometer_SMD:Potentiometer_Vishay_TS53YJ_Vertical; symbol Device:R_POT_Small -> Device:R_Potentiometer_Small
- SW1: renamed from SW2; footprint (none) -> Button_Switch_SMD:SW_SPST_B3S-1000
- SW2: renamed from SW5; footprint (none) -> SP3T_THT:MHS133G04
- U4, U5: footprint N16 -> Package_SO:SOIC-16W_5.3x10.2mm_P1.27mm; symbol 74hc138:SN74HC138N -> 74HC138:SN74HC138N
- U6: footprint (none) -> Package_SO:SOIC-14_3.9x8.7mm_P1.27mm
- renumbered X8.000Mhz1 to CLK2, R3 to R5
Connections:
- net +5V: now also A1.4 (3V3), CPU1.6 (VCC), J2.19 (Pin_19), J2.20 (Pin_20), R15.2, R16.1, R18.2, J3.19 (Pin_19), J3.20 (Pin_20), RN1.1 (common), U10.26 (VCC), U8.14 (VDD); no longer A1.5 (+5V), CPU1.11 (VCC), J2.10 (Pin_10)
- net A0: now also CPU1.27 (A0), J2.36 (Pin_36), J3.36 (Pin_36), U10.9 (A0); no longer CPU1.30 (A0), J2.18 (Pin_18)
- net A1: now also CPU1.28 (A1), J2.35 (Pin_35), J3.35 (Pin_35), U10.8 (A1); no longer CPU1.31 (A1), J2.19 (Pin_19)
- net A10: now also CPU1.38 (A10), J2.26 (Pin_26), J3.26 (Pin_26); no longer CPU1.40 (A10), J2.28 (Pin_28)
- net A11: now also CPU1.40 (A11), J2.25 (Pin_25), J3.25 (Pin_25); no longer CPU1.1 (A11), J2.29 (Pin_29)
- net A12: now also CPU1.41 (A12), J2.24 (Pin_24), J3.24 (Pin_24); no longer CPU1.2 (A12), J2.30 (Pin_30)
- net A13: now also CPU1.42 (A13), J2.23 (Pin_23), J3.23 (Pin_23), RN7.7 (R6); no longer CPU1.3 (A13), J2.31 (Pin_31)
- net A14: now also CPU1.43 (A14), J2.22 (Pin_22), J3.22 (Pin_22), RN7.8 (R7); no longer CPU1.4 (A14), J2.32 (Pin_32)
- net A15: now also CPU1.44 (A15), J2.21 (Pin_21), J3.21 (Pin_21), RN7.9 (R8); no longer CPU1.5 (A15), J2.9 (Pin_9)
- net A2: now also CPU1.29 (A2), J2.34 (Pin_34), J3.34 (Pin_34); no longer CPU1.32 (A2), J2.20 (Pin_20)
- net A3: now also CPU1.30 (A3), J2.33 (Pin_33), J3.33 (Pin_33); no longer CPU1.33 (A3), J2.21 (Pin_21)
- net A4: now also CPU1.31 (A4), J2.32 (Pin_32), J3.32 (Pin_32); no longer CPU1.34 (A4), J2.22 (Pin_22)
- net A5: now also CPU1.32 (A5), J2.31 (Pin_31), J3.31 (Pin_31); no longer CPU1.35 (A5), J2.23 (Pin_23)
- net A6: now also CPU1.34 (A6), J2.30 (Pin_30), J3.30 (Pin_30); no longer CPU1.36 (A6), J2.24 (Pin_24)
- net A7: now also CPU1.35 (A7), J2.29 (Pin_29), J3.29 (Pin_29); no longer CPU1.37 (A7), J2.25 (Pin_25)
- net A8: now also CPU1.36 (A8), J2.28 (Pin_28), J3.28 (Pin_28); no longer CPU1.38 (A8), J2.26 (Pin_26)
- net A9: now also CPU1.37 (A9), J3.27 (Pin_27); no longer CPU1.39 (A9)
- net BUSACK: now also A1.5 (A3), CPU1.20 (~{BUSACK}), D28.2 (A); no longer CPU1.23 (~{BUSACK})
- net BUSRQ: now also A1.12 (D10), CPU1.22 (~{BUSRQ}), D27.2 (A), RN1.2 (R1); no longer CPU1.25 (~{BUSRQ})
- net Clock: now also CPU1.1 (~{CLK}), D1.1 (K), D3.1 (K), D7.1 (K), R4.1; no longer CPU1.6 (~{CLK}), D2.1 (K), D4.1 (K), D8.1 (K)
- net D0: now also A1.20 (D2), CPU1.9 (D0), J3.8 (Pin_8), U10.34 (D0); no longer A1.17 (D2/SDA), CPU1.14 (D0)
- net D1: now also A1.19 (D3), CPU1.10 (D1), J3.7 (Pin_7), U10.33 (D1); no longer A1.18 (D3/SCL), CPU1.15 (D1)
- net D2: now also A1.18 (D4), CPU1.7 (D2), J3.6 (Pin_6), U10.32 (D2); no longer A1.19 (D4), CPU1.12 (D2)
- net D3: now also A1.17 (D5), CPU1.3 (D3), J3.5 (Pin_5), U10.31 (D3); no longer A1.20 (D5), CPU1.8 (D3)
- net D4: now also A1.16 (D6), CPU1.2 (D4), J3.4 (Pin_4), U10.30 (D4); no longer A1.21 (D6), CPU1.7 (D4)
- net D5: now also A1.15 (D7), CPU1.4 (D5), J3.3 (Pin_3), U10.29 (D5); no longer A1.22 (D7), CPU1.9 (D5)
- net D6: now also A1.14 (D8), CPU1.5 (D6), J3.2 (Pin_2), U10.28 (D6); no longer A1.23 (D8), CPU1.10 (D6)
- net D7: now also A1.13 (D9), CPU1.8 (D7), J3.1 (Pin_1), U10.27 (D7); no longer A1.24 (D9), CPU1.13 (D7)
- net GND: now also A1.2 (GND), A1.21 (GND), A1.22 (GND), CPU1.26 (GND), J2.39 (Pin_39), J2.40 (Pin_40), R14.2, C8.1, J3.39 (Pin_39), J3.40 (Pin_40), R10.2, R3.2, R4.2, RN2.1 (common), RN3.1 (common), RN4.1 (common), RN5.1 (common), RN6.1 (common), RN7.1 (common), SW3.1, U10.7 (GND), U8.7 (VSS); no longer A1.6 (GND), CPU1.29 (GND), J2.16 (Pin_16), J2.17 (Pin_17), R14.1, R16.1, R18.1
- net HALT: now also CPU1.14 (~{HALT}), D26.2 (A); no longer CPU1.18 (~{HALT})
- net INT: now also CPU1.12 (~{INT}), D22.2 (A), J2.14 (Pin_14), J3.14 (Pin_14), RN1.5 (R4); no longer CPU1.16 (~{INT})
- net IORQ: now also CPU1.16 (~{IORQ}), J2.10 (Pin_10), D32.2 (A), J3.10 (Pin_10), RN1.6 (R5); no longer CPU1.20 (~{IORQ}), J2.12 (Pin_12)
- net M1: now also CPU1.24 (~{M1}), D23.2 (A); no longer CPU1.27 (~{M1})
- net MREQ: now also CPU1.15 (~{MREQ}), J2.11 (Pin_11), D31.2 (A), J3.11 (Pin_11), RN7.2 (R1); no longer CPU1.19 (~{MREQ}), J2.13 (Pin_13)
- net NMI: now also CPU1.13 (~{NMI}), D21.2 (A), J2.15 (Pin_15), J3.15 (Pin_15), RN1.4 (R3); no longer CPU1.17 (~{NMI})
- net RAM1-CS: now also U8.11; no longer D21.1 (K)
- net RD: now also A1.8 (A0), CPU1.18 (~{RD}), J2.12 (Pin_12), D30.2 (A), J3.12 (Pin_12), U10.5 (~{RD}); no longer A1.9 (A0), CPU1.21 (~{RD}), J2.14 (Pin_14)
- net RFSH: now also CPU1.25 (~{RFSH}), D24.2 (A); no longer CPU1.28 (~{RFSH})
- net ROM1-CS: now also U1.11; no longer D22.1 (K), D23.1 (K)
- net RST: now also CPU1.23 (~{RESET}), J2.9 (Pin_9), C8.2, D33.2 (A), J3.9 (Pin_9), SW3.2; no longer A1.25 (D10), J2.11 (Pin_11), U2.13 (~{OE}), U3.13 (~{OE})
- net WAIT: now also CPU1.21 (~{WAIT}), J2.16 (Pin_16), D25.2 (A), J3.16 (Pin_16), RN1.3 (R2); no longer CPU1.24 (~{WAIT})
- net WR: now also CPU1.19 (~{WR}), J2.13 (Pin_13), D29.2 (A), J3.13 (Pin_13), U10.36 (~{WR}); no longer A1.10 (A1), CPU1.22 (~{WR}), J2.15 (Pin_15), ROM1.27 (~{WE})
- net at U2.11 (SRCLK), U3.11 (SRCLK): now also A1.10 (D14); no longer A1.27 (D14)
- net at U2.12 (RCLK), U3.12 (RCLK): now also A1.11 (D16); no longer A1.26 (D16)
- net at U2.14 (SER): now also A1.9 (D15); no longer A1.28 (D15)
- net PROG-WR: now reaches A1.7 (A1)
- net PROG-WR: now also R16.2, ROM1.27 (~{WE})
- net at D41.1 (K): now also RN5.9 (R8)
- net at D17.1 (K): now also RN2.6 (R5)
- net at D14.1 (K): now also RN2.3 (R2)
- net at R2.2, U1.2: now also D2.2 (A), SW2.2; no longer SW2.1
- net at U1.3: now also D1.2 (A); no longer D2.2 (A)
- net at D43.1 (K): now also RN6.3 (R2)
- net at U7.1 (PA3): now also J4.8 (Pin_8)
- net at U7.10 (PC7): now also J6.7 (Pin_7)
- net at U7.11 (PC6): now also J6.5 (Pin_5)
- net at U7.12 (PC5): now also J6.3 (Pin_3)
- net at U7.13 (PC4): now also J6.1 (Pin_1)
- net at U7.14 (PC0): now also J6.2 (Pin_2)
- net at U7.15 (PC1): now also J6.4 (Pin_4)
- net at U7.16 (PC2): now also J6.6 (Pin_6)
- net at U7.17 (PC3): now also J6.8 (Pin_8)
- net at U7.18 (PB0): now also J5.2 (Pin_2)
- net at U7.19 (PB1): now also J5.4 (Pin_4)
- net at U7.2 (PA2): now also J4.6 (Pin_6)
- net at U7.20 (PB2): now also J5.6 (Pin_6)
- net at U7.21 (PB3): now also J5.8 (Pin_8)
- net at U7.22 (PB4): now also J5.1 (Pin_1)
- net at U7.23 (PB5): now also J5.3 (Pin_3)
- net at U7.24 (PB6): now also J5.5 (Pin_5)
- net at U7.25 (PB7): now also J5.7 (Pin_7)
- net at U7.3 (PA1): now also J4.4 (Pin_4)
- net RST-INV: now reaches U6.2, U7.35 (RESET)
- net RST-INV: now also R18.1, U10.35 (RESET)
- net at U7.37 (PA7): now also J4.7 (Pin_7)
- net at U7.38 (PA6): now also J4.5 (Pin_5)
- net at U7.39 (PA5): now also J4.3 (Pin_3)
- net at U7.4 (PA0): now also J4.2 (Pin_2)
- net at U7.40 (PA4): now also J4.1 (Pin_1)
- net EXT-IO4-CS: now reaches U5.10 (Y5)
- net EXT-IO4-CS: now also J3.18 (Pin_18)
- net EXT-IO3-CS: now reaches U5.11 (Y4)
- net EXT-IO3-CS: now also J2.38 (Pin_38)
- net EXT-IO2-CS: now reaches U5.12 (Y3)
- net EXT-IO2-CS: now also J2.17 (Pin_17)
- net EXT-IO1-CS: now reaches U5.13 (Y2)
- net EXT-IO1-CS: now also J2.18 (Pin_18)
- net IO2-CS: now reaches U5.14 (Y1)
- net IO2-CS: now also U10.6 (~{CS})
- net EXT-IO6-CS: now reaches U5.7 (Y7)
- net EXT-IO6-CS: now also J3.38 (Pin_38)
- net EXT-IO5-CS: now reaches U5.9 (Y6)
- net EXT-IO5-CS: now also J3.17 (Pin_17)
- net at U1.10: now also D7.2 (A); no longer D8.2 (A)
- net at R13.2, SW2.4, U1.9: now also D8.2 (A)
- net at D45.1 (K): now also RN6.5 (R4)
- net at D48.1 (K): now also RN6.8 (R7)
- net at D46.1 (K): now also RN6.6 (R5)
- net at U4.14 (Y1): now also U1.12; no longer D22.2 (A)
- net at D13.1 (K): now also RN2.2 (R1)
- net at D39.1 (K): now also RN5.7 (R6)
- net at D40.1 (K): now also RN5.8 (R7); no longer R18.2
- net at U4.10 (Y5): now also U8.8
- net at U4.11 (Y4): now also U8.9
- net at U4.12 (Y3): now also U8.12
- net at U4.13 (Y2): now also U8.13; no longer D21.2 (A)
- net at U4.15 (Y0): now also U1.13; no longer D23.2 (A)
- net at U4.7 (Y7): now also U8.5
- net at U4.9 (Y6): now also U8.6
- net at D15.1 (K): now also RN2.4 (R3)
- net at D4.2 (A): now also R7.2, SW2.3, U1.6; no longer U1.4
- net at D42.1 (K): now also RN6.2 (R1)
- net at D36.1 (K): now also RN5.4 (R3); no longer R14.2
- net at D34.1 (K): now also RN5.2 (R1)
- net at R8.2: now also SW2.1; no longer SW2.3
- net at D35.1 (K): now also RN5.3 (R2)
- net at D18.1 (K): now also RN2.7 (R6)
- net at D44.1 (K): now also RN6.4 (R3)
- net at D38.1 (K): now also RN5.6 (R5); no longer R16.2
- net at D19.1 (K): now also RN2.8 (R7)
- net at D37.1 (K): now also RN5.5 (R4)
- net at D49.1 (K): now also RN6.9 (R8)
- net at D16.1 (K): now also RN2.5 (R4)
- net at D20.1 (K): now also RN2.9 (R8)
- net at D47.1 (K): now also RN6.7 (R6)
- new net: A1.6 (A2), U2.13 (~{OE}), U3.13 (~{OE})
- new net: D33.1 (K), RN4.2 (R1)
- new net: D32.1 (K), RN4.3 (R2)
- new net: D31.1 (K), RN4.4 (R3)
- new net: D30.1 (K), RN4.5 (R4)
- new net: D29.1 (K), RN4.6 (R5)
- new net: D28.1 (K), RN4.7 (R6)
- new net: D27.1 (K), RN4.8 (R7)
- new net: D26.1 (K), RN4.9 (R8)
- new net: J7.1 (Pin_1), U10.40 (PA4)
- new net: J7.2 (Pin_2), U10.4 (PA0)
- new net: J7.3 (Pin_3), U10.39 (PA5)
- new net: J7.4 (Pin_4), U10.3 (PA1)
- new net: J7.5 (Pin_5), U10.38 (PA6)
- new net: J7.6 (Pin_6), U10.2 (PA2)
- new net: J7.7 (Pin_7), U10.37 (PA7)
- new net: J7.8 (Pin_8), U10.1 (PA3)
- new net: D23.1 (K), RN3.4 (R3)
- new net: D25.1 (K), RN3.2 (R1)
- new net: D24.1 (K), RN3.3 (R2)
- new net: D22.1 (K), RN3.5 (R4)
- new net: D21.1 (K), RN3.6 (R5)
- new net: J9.1 (Pin_1), U10.13 (PC4)
- new net: J9.2 (Pin_2), U10.14 (PC0)
- new net: J9.3 (Pin_3), U10.12 (PC5)
- new net: J9.4 (Pin_4), U10.15 (PC1)
- new net: J9.5 (Pin_5), U10.11 (PC6)
- new net: J9.6 (Pin_6), U10.16 (PC2)
- new net: J9.7 (Pin_7), U10.10 (PC7)
- new net: J9.8 (Pin_8), U10.17 (PC3)
- new net: U8.10, U8.2
- new net: U8.1, U8.4
- new net: D4.1 (K), R10.1
- new net: J8.2 (Pin_2), U10.18 (PB0)
- new net: J8.4 (Pin_4), U10.19 (PB1)
- new net: J8.6 (Pin_6), U10.20 (PB2)
- new net: J8.8 (Pin_8), U10.21 (PB3)
- new net: J8.1 (Pin_1), U10.22 (PB4)
- new net: J8.3 (Pin_3), U10.23 (PB5)
- new net: J8.5 (Pin_5), U10.24 (PB6)
- new net: J8.7 (Pin_7), U10.25 (PB7)
- new net: D3.2 (A), U1.4
- new net: D8.1 (K), R14.1
- new net: D2.1 (K), R3.1
- new net EXT-CS: J2.37 (Pin_37), J3.37 (Pin_37), U8.3
- no-connect marks 30 -> 26
Other:
- removed sheet Flash Cartridge
- note added: "Power Connector"
- moved on the sheet: D13, D14, D15, D16, D17, D18, D19, D2, D20, D34, D35, D36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

Commit message: Schematic cahnges, PCB changes, test asm changes
Parts:
- removed D1, D3, D7: D, symbol Device:D_Small
- removed R4: 10K, Resistor_SMD:R_0603_1608Metric, symbol Device:R_Small
- added U9: 74LS32, Capacitor_SMD:C_1206_3216Metric, symbol 74xx:74LS32
- C1, C8: footprint Capacitor_SMD:C_0603_1608Metric -> Capacitor_SMD:C_1206_3216Metric
- RAM1: footprint Package_DIP:DIP-28_W15.24mm_Socket -> Package_SO:TSOP-I-28_11.8x8mm_P0.55mm
Connections:
- net +5V: now also U9.14 (VCC); no longer R18.2
- net Clock: now also U9.6
- net EXT-CS: now also U1.11; no longer U8.3
- net GND: now also R18.2, U9.7 (GND)
- net IORQ: now also U9.9; no longer RN1.6 (R5), U4.6 (G1), U5.4 (~{G2A})
- net RAM1-CS: now also U4.14 (Y1); no longer U8.11
- net ROM1-CS: now also U4.15 (Y0); no longer U1.11
- net PROG-OE: now reaches A1.6 (A2), U2.13 (~{OE}), U3.13 (~{OE})
- net PROG-OE: now also U6.3
- net FstOUT: now reaches U1.3
- net FstOUT: now also U9.5
- net ManOUT: now reaches U1.10
- net ManOUT: now also U9.1
- net at U1.12: now also U8.3; no longer U4.14 (Y1)
- net at U1.13: now also U8.11; no longer U4.15 (Y0)
- net AdjOUT: now reaches U1.4
- net AdjOUT: now also U9.2
- net at U6.4: now also U9.10
- new net: U9.3, U9.4
- new net IOREQ: U4.6 (G1), U5.4 (~{G2A}), U9.8
- no-connect marks 26 -> 32
Other:
- moved on the sheet: D2, D4, D8, R10, R14, R3, SW2, U1A, U1B, U1C, U1D, U1E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

Commit message: Board revision 1
Parts:
- A1: footprint (none) -> Package_DIP:DIP-24_W15.24mm_Socket
- U9: footprint Capacitor_SMD:C_1206_3216Metric -> Package_SO:SOIC-14_3.9x8.7mm_P1.27mm
Other:
- moved on the sheet: D13, D14, D15, D16, D17, D18, D19, D20, D21, D22, D23, D24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

Commit message: Schematic/code changes, updated to 2024
Parts:
- added C10, C9: 22pF, Capacitor_SMD:C_0603_1608Metric, symbol Device:C_Small
- added C11, C12: 1uF, Capacitor_SMD:C_0603_1608Metric, symbol Device:C_Small
- added CLK3: 16MHz, symbol Device:Crystal
- added D1, D3: LED_Red, LED_SMD:LED_0603_1608Metric, symbol Device:LED_Small
- added J10: Conn_02x03_Counter_Clockwise, Connector_PinHeader_2.54mm:PinHeader_2x03_P2.54mm_Vertical, symbol Connector_Generic:Conn_02x03_Odd_Even
- added J11: USB_C_Receptacle_USB2.0, Connector_USB:USB_C_Receptacle_Palconn_UTC16-G, symbol Connector:USB_C_Receptacle_USB2.0
- added R17, R19: 22R, Resistor_SMD:R_0603_1608Metric, symbol Device:R_Small
- added R20, R4: 10K, Resistor_SMD:R_0603_1608Metric, symbol Device:R_Small
- added R21, R22: 1K, Resistor_SMD:R_0603_1608Metric, symbol Device:R_Small
- added U11: ATmega32U4RC-A, Package_QFP:TQFP-44_10x10mm_P0.8mm, symbol MCU_Microchip_ATmega:ATmega32U4RC-A
- C8: footprint Capacitor_SMD:C_1206_3216Metric -> Capacitor_SMD:C_0603_1608Metric
- CLK2: footprint Oscillator:Oscillator_DIP-14 -> (none)
Connections:
- net +5V: now also D1.2 (A), D3.2 (A), J10.2 (Pin_2), R20.2, R4.1, U11.14 (VCC), U11.24 (AVCC), U11.34 (VCC), U11.44 (AVCC)
- net BUSACK: now also U11.39 (PF4(A3))
- net BUSRQ: now also U11.30 (PB6(D10))
- net D0: now also U11.19 (PD1(D2))
- net D1: now also U11.18 (PD0(D3))
- net D2: now also U11.25 (PD4(D4))
- net D3: now also U11.31 (PC6(D5))
- net D4: now also U11.27 (PD7(D6))
- net D5: now also U11.1 (PE6(D7))
- net D6: now also U11.28 (PB4(D8))
- net D7: now also U11.29 (PB5(D9))
- net GND: now also C10.2, C11.2, C12.1, C9.2, J10.6 (Pin_6), J11.A1 (GND), J11.A12 (GND), J11.B1 (GND), J11.B12 (GND), J11.S1 (SHIELD), U11.15 (GND), U11.23 (GND), U11.33 (~{HWB}/PE2), U11.35 (GND), U11.43 (GND), U11.5 (UGND)
- net PROG-OE: now also R20.1, U11.38 (PF5(A2))
- net PROG-WR: now also U11.37 (PF6(A1))
- net RD: now also U11.36 (PF7(A0))
- net at D2.2 (A), R2.2, U1.2: now also SW2.1; no longer SW2.2
- net at R8.2: now also SW2.2; no longer SW2.1
- new net: R17.2, U11.4 (D+)
- new net: D1.1 (K), R21.1
- new net: C11.1, U11.6 (UCAP)
- new net: C10.1, CLK3.1, U11.16 (XTAL2)
- new net: C9.1, CLK3.2, U11.17 (XTAL1)
- new net: R22.2, U11.22 (PD5)
- new net: R19.2, U11.3 (D-)
- new net: R21.2, U11.8 (PB0)
- new net: D3.1 (K), R22.1
- new net MISO: J10.1 (Pin_1), U11.11 (PB3(D14/MISO))
- new net MOSI: J10.4 (Pin_4), U11.10 (PB2(D16/MOSI))
- new net ProgReset: J10.5 (Pin_5), R4.2, U11.13 (~{RESET})
- new net SPISCK: J10.3 (Pin_3), U11.9 (PB1(D15/SCK))
- new net USB-D+: J11.A6 (D+), J11.B6 (D+), R17.1
- new net USB-D-: J11.A7 (D-), J11.B7 (D-), R19.1
- new net VBUS: C12.2, J11.A4 (VBUS), J11.A9 (VBUS), J11.B4 (VBUS), J11.B9 (VBUS), U11.2 (UVCC), U11.7 (VBUS)
- no-connect marks 32 -> 37
Other:
- note added: "Indicator LEDs"
- note added: "Logic Power"
- moved on the sheet: J2, J3, J4, J5, J6, J7, J8, J9, R18, U10, U1E, U5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

Commit message: schematic updates, assembly progress
Parts:
- added D10, D11, D12, D50, D7, D9: LED_Green, LED_SMD:LED_0603_1608Metric, symbol Device:LED_Small
- added RN8: EXB-D10C102J, r_network:EXB-D10C103J, symbol Device:R_Network08
- C1: footprint Capacitor_SMD:C_1206_3216Metric -> Capacitor_SMD:C_0603_1608Metric
- CLK2: footprint (none) -> Oscillator:Oscillator_DIP-14
- renumbered RN7 to RN2, RN2 to RN3, RN3 to RN4, RN4 to RN5, RN5 to RN6, RN6 to RN7
Connections:
- net EXT-CS: now also U8.3, D11.2 (A); no longer U1.11
- net GND: now also RN8.1 (common); no longer J2.39 (Pin_39), J3.39 (Pin_39)
- net IO1-CS: now also D12.2 (A)
- net IO2-CS: now also D50.2 (A)
- net RAM1-CS: now also D9.2 (A)
- net ROM1-CS: now also D7.2 (A)
- net at U1.13: no longer U8.11
- net at U1.12: no longer U8.3
- new net: D7.1 (K), RN8.4 (R3)
- new net: D9.1 (K), RN8.5 (R4)
- new net: D10.1 (K), RN8.6 (R5)
- new net: D11.1 (K), RN8.7 (R6)
- new net: D12.1 (K), RN8.8 (R7)
- new net: D50.1 (K), RN8.9 (R8)
- new net EXT-CS2: D10.2 (A), J2.39 (Pin_39), J3.39 (Pin_39), U8.11
- no-connect marks 37 -> 43
Other:
- note added: "8KiB offset: 0B"
- note added: "8KiB offset: 8KiB"
- note removed: "8KB offset: 0B"
- note removed: "8KB offset: 8KB"
- moved on the sheet: C10, C11, C12, C9, CLK3, D1, D3, J10, J11, R17, R19, R21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
