File: z80/z80.kicad_sch (KiCad schematic)
At the start: 125 parts, among them J1 PinHeader_Female01x02, J10 Conn_02x03_Counter_Clockwise, J11 USB_C_Receptacle_USB2.0, J2 PinHeader_Female16x02, J3 PinHeader_Female16x02, J4 PinHeader_Female04x02, J5 PinHeader_Female04x02, J6 PinHeader_Female04x02, J7 PinHeader_Female04x02, J8 PinHeader_Female04x02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

Commit message: finished v2 of hardware, updated eeprom prog pins
Parts:
- removed A1: 32U4 Arduino, Package_DIP:DIP-24_W15.24mm_Socket, symbol promicro:Sparkfun_Pro_Micro
- CLK3: footprint (none) -> Crystal:Crystal_HC49-U_Vertical
- J11: footprint Connector_USB:USB_C_Receptacle_Palconn_UTC16-G -> Connector_USB:USB_C_Receptacle_GCT_USB4085
Connections:
- net VBUS is gone; now on net +5V: C12.2, J11.A4 (VBUS), J11.A9 (VBUS), J11.B4 (VBUS), J11.B9 (VBUS), U11.2 (UVCC), U11.7 (VBUS)
- net SRCLK: now reaches U2.11 (SRCLK), U3.11 (SRCLK)
- net SRCLK: now also U11.26 (PD6(D12))
- net RCLK: now reaches U2.12 (RCLK), U3.12 (RCLK)
- net RCLK: now also U11.12 (PB7(D11))
- net SER: now reaches U2.14 (SER)
- net SER: now also U11.32 (PC7(D13))
- no-connect marks 43 -> 40
Other:
- moved on the sheet: C10, C11, C12, C9, CLK3, D1, D10, D11, D12, D13, D14, D15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
