File: z80/_autosave-z80.kicad_sch (KiCad schematic)
At the start: 115 parts, among them J1 Screw_Terminal_01x02, J2 Conn_02x16_Counter_Clockwise, SW11 SW_SPDT, SW13 SW_DPDT_x2, SW3 SW_SPDT, SW4 SW_Push, SW7 SW_SPST, SW8 SW_SP3T, U1 4081, U11 4069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

Commit message: hoi
Parts:
- J1: footprint (none) -> TerminalBlock_4Ucon:TerminalBlock_4Ucon_1x02_P3.50mm_Horizontal
- gave numbers to parts that had none: 2
- renumbered R5 to R10, R3 to R2, R6 to R3, R7 to R4, R42 to R40, R43 to R41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
