File: z80/FlashCartridge.kicad_sch (KiCad schematic)
At the start: 5 parts

Commit message: schematic changes
Parts:
- gave numbers to parts that had none: 5
Changed lines of the file:
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@@
   (title_block
     (title "z80 Flash Cartridge")
-    (date "2022-11-06")
-    (rev "1.6")
+    (date "2023-02-27")
+    (rev "1.7")
     (company "T. van de Weg")
   )
@@
   (symbol (lib_id "Device:R_Small") (at 90.17 95.885 270) (unit 1)
     (in_bom yes) (on_board yes)
-    (property "Reference" "R?" (id 0) (at 90.17 100.8634 90)
+    (property "Reference" "R37" (id 0) (at 90.17 100.8634 90)
       (effects (font (size 1.27 1.27)) hide)
     )
@@
   (symbol (lib_id "74xx:74LS174") (at 72.39 93.345 0) (unit 1)
     (in_bom yes) (on_board yes)
-    (property "Reference" "U?" (id 0) (at 66.04 79.375 0))
+    (property "Reference" "U8" (id 0) (at 66.04 79.375 0))
     (property "Value" "74LS174" (id 1) (at 77.47 79.375 0))
     (property "Footprint" "Package_SO:SO-16_5.3x10.2mm_P1.27mm" (id 2) (at 72.39 93.345 0)
@@
   (symbol (lib_id "Device:R_Small") (at 59.69 108.585 0) (unit 1)
     (in_bom yes) (on_board yes)
-    (property "Reference" "R?" (id 0) (at 64.6684 108.585 90)
+    (property "Reference" "R36" (id 0) (at 64.6684 108.585 90)
       (effects (font (size 1.27 1.27)) hide)
     )
@@
   (symbol (lib_id "Connector_Generic:Conn_02x16_Counter_Clockwise") (at 105.41 126.365 270) (unit 1)
     (in_bom yes) (on_board yes)
-    (property "Reference" "J?" (id 0) (at 82.8802 126.4666 90)
+    (property "Reference" "J3" (id 0) (at 82.8802 126.4666 90)
       (effects (font (size 1.27 1.27)) (justify right) hide)
     )
@@
   (symbol (lib_id "Memory_Flash:SST39SF040") (at 107.95 75.565 0) (unit 1)
     (in_bom yes) (on_board yes)
-    (property "Reference" "U?" (id 0) (at 116.84 42.545 0))
+    (property "Reference" "U9" (id 0) (at 116.84 42.545 0))
     (property "Value" "SST39SF040" (id 1) (at 100.33 42.545 0))
     (property "Footprint" "Package_DIP:DIP-32_W15.24mm_Socket" (id 2) (at 107.95 67.945 0)

Commit message: Schematic changes, test script
Parts:
- R38: renamed from R36; footprint Resistor_SMD:R_0603_1608Metric_Pad0.98x0.95mm_HandSolder -> Resistor_SMD:R_0603_1608Metric
- R39: renamed from R37; footprint Resistor_SMD:R_0603_1608Metric_Pad0.98x0.95mm_HandSolder -> Resistor_SMD:R_0603_1608Metric
