File: z80/z80.kicad_pcb (KiCad board)
At the start: 2 copper layers, 224.2 x 181 mm, 108 parts, among them J1 Conn_02x16_Counter_Clockwise, J2 Conn_02x16_Counter_Clockwise, SW10 SW_DIP_x08, SW12 SW_DIP_x08, SW13 SW_DIP_x08, SW14 SW_DIP_x08, SW5 SW_DIP_x08, SW9 SW_DIP_x08, U1 4081, U14 74LS174, U15 74LS174, U2 74HC595, U20 74LS174, U23 SST39SF040, U24 74LS174, U25 74LS174, U3 74HC595, X8.000Mhz1 TFT680

Commit message: hoi
Parts:
- removed SW10, SW12, SW9: SW_DIP_x08, Button_Switch_THT:SW_DIP_SPSTx08_Piano_10.8x21.88mm_W7.62mm_P2.54mm
- added J1: Screw_Terminal_01x02, TerminalBlock_4Ucon:TerminalBlock_4Ucon_1x02_P3.50mm_Horizontal, F.Cu at (61.0, 0.64)
- added J3: Conn_02x16_Counter_Clockwise, Connector_PinHeader_2.54mm:PinHeader_2x16_P2.54mm_Horizontal, F.Cu at (-7.78, -1.47)
- added R50: 1K, Resistor_SMD:R_0603_1608Metric_Pad0.98x0.95mm_HandSolder, F.Cu at (8.02, 39.8)
- added R51: 1K, Resistor_SMD:R_0603_1608Metric_Pad0.98x0.95mm_HandSolder, F.Cu at (-7.93, 40.2)
- added U19: 74LS174, Package_SO:SO-16_5.3x10.2mm_P1.27mm, F.Cu at (30.5, 2.08)
- added U20: SST39SF040, Package_DIP:DIP-32_W15.24mm_Socket, F.Cu at (7.92, -1.67)
- renumbered J1 to J2, R5 to R10, R3 to R2, R6 to R3, R7 to R4, R42 to R40, R43 to R41, R44 to R42, R45 to R43, R46 to R44, R47 to R45, R48 to R46, R49 to R47, R50 to R48, R51 to R49, R4 to R5, R2 to R6, R8 to R7, R9 to R8, R10 to R9, U15 to U10, U24 to U17, U25 to U18, U14 to U9
Connections:
- net A13 renamed /A13
- net A14 renamed /A14
- net Net-(RAM1-Pad20) renamed /RAM1-CS
- net Net-(ROM1-Pad20) renamed /ROM1-CS
- A1 pad 17: Net-(A1-Pad17) -> unconnected-(A1-Pad17)
- A1 pad 18: Net-(A1-Pad18) -> unconnected-(A1-Pad18)
- A1 pad 19: Net-(A1-Pad19) -> unconnected-(A1-Pad19)
- A1 pad 20: Net-(A1-Pad20) -> unconnected-(A1-Pad20)
- A1 pad 21: Net-(A1-Pad21) -> unconnected-(A1-Pad21)
- A1 pad 22: Net-(A1-Pad22) -> unconnected-(A1-Pad22)
- A1 pad 23: Net-(A1-Pad23) -> unconnected-(A1-Pad23)
- A1 pad 24: Net-(A1-Pad24) -> unconnected-(A1-Pad24)
- A1 pad 5: Net-(A1-Pad5) -> unconnected-(A1-Pad5)
- CPU1 pad 1: A11 -> /A11
- CPU1 pad 18: unconnected-(CPU1-Pad18) -> /HALT
- CPU1 pad 2: A12 -> /A12
- CPU1 pad 21: RD -> /RD
- CPU1 pad 22: WR -> /WR
- CPU1 pad 24: unconnected-(CPU1-Pad24) -> /WAIT
- CPU1 pad 27: unconnected-(CPU1-Pad27) -> /M1
- CPU1 pad 28: unconnected-(CPU1-Pad28) -> /RFSH
- CPU1 pad 34: A4 -> /A4
- CPU1 pad 35: A5 -> /A5
- CPU1 pad 36: A6 -> /A6
- CPU1 pad 37: A7 -> /A7
- CPU1 pad 38: A8 -> /A8
- CPU1 pad 39: A9 -> /A9
- CPU1 pad 40: A10 -> /A10
- CPU1 pad 5: A15 -> /A15
- D10 pad 2: A7 -> /A7
- D11 pad 2: A8 -> /A8
- D12 pad 2: A9 -> /A9
- D13 pad 2: A10 -> /A10
- D14 pad 2: A11 -> /A11
- D15 pad 2: A12 -> /A12
- D18 pad 2: A15 -> /A15
- D7 pad 2: A4 -> /A4
- D8 pad 2: A5 -> /A5
- D9 pad 2: A6 -> /A6
- J2 pad 14: RD -> /RD
- J2 pad 15: WR -> /WR
- J2 pad 22: A4 -> /A4
- J2 pad 23: A5 -> /A5
- J2 pad 24: A6 -> /A6
- J2 pad 25: A7 -> /A7
- J2 pad 26: A8 -> /A8
- J2 pad 27: A9 -> /A9
- J2 pad 28: A10 -> /A10
- J2 pad 29: A11 -> /A11
- J2 pad 30: A12 -> /A12
- J2 pad 9: A15 -> /A15
- RAM1 pad 2: A12 -> /A12
- RAM1 pad 21: A10 -> /A10
- RAM1 pad 22: RD -> /RD
- RAM1 pad 23: A11 -> /A11
- RAM1 pad 24: A9 -> /A9
- RAM1 pad 25: A8 -> /A8
- RAM1 pad 27: WR -> /WR
- RAM1 pad 3: A7 -> /A7
- RAM1 pad 4: A6 -> /A6
- RAM1 pad 5: A5 -> /A5
- RAM1 pad 6: A4 -> /A4
- ROM1 pad 1: unconnected-(ROM1-Pad1) -> (no net)
- ROM1 pad 10: PA0 -> A0
- ROM1 pad 11: PD0 -> D0
- ROM1 pad 12: PD1 -> D1
- ROM1 pad 13: PD2 -> D2
- ROM1 pad 15: PD3 -> D3
- ROM1 pad 16: PD4 -> D4
- ROM1 pad 17: PD5 -> D5
- ROM1 pad 18: PD6 -> D6
- ROM1 pad 19: PD7 -> D7
- ROM1 pad 2: PA12 -> /A12
- ROM1 pad 21: PA10 -> /A10
- ROM1 pad 22: PRD -> /RD
- ROM1 pad 23: PA11 -> /A11
- ROM1 pad 24: PA9 -> /A9
- ROM1 pad 25: PA8 -> /A8
- ROM1 pad 26: unconnected-(ROM1-Pad26) -> (no net)
- ROM1 pad 27: PWR -> /WR
- ROM1 pad 3: PA7 -> /A7
- ROM1 pad 4: PA6 -> /A6
- ROM1 pad 5: PA5 -> /A5
- ROM1 pad 6: PA4 -> /A4
- ROM1 pad 7: PA3 -> A3
- ROM1 pad 8: PA2 -> A2
- ROM1 pad 9: PA1 -> A1
- U2 pad 1: Net-(SW13-Pad2) -> A1
- U2 pad 15: Net-(SW13-Pad1) -> A0
- U2 pad 2: Net-(SW13-Pad3) -> A2
- U2 pad 3: Net-(SW13-Pad4) -> A3
- U2 pad 4: Net-(SW13-Pad5) -> /A4
- U2 pad 5: Net-(SW13-Pad6) -> /A5
- U2 pad 6: Net-(SW13-Pad7) -> /A6
- U2 pad 7: Net-(SW13-Pad8) -> /A7
- U3 pad 1: Net-(SW14-Pad2) -> /A9
- U3 pad 15: Net-(SW14-Pad1) -> /A8
- U3 pad 2: Net-(SW14-Pad3) -> /A10
- U3 pad 3: Net-(SW14-Pad4) -> /A11
- U3 pad 4: Net-(SW14-Pad5) -> /A12
Routing:
- net A11: track 95.9 -> 0.00 mm, vias 2 -> 0
- net /A11: track 0.00 -> 95.9 mm, vias 0 -> 2
- net A12: track 90.0 -> 0.00 mm, vias 1 -> 0
- net /A12: track 0.00 -> 90.0 mm, vias 0 -> 1
- net A8: track 86.2 -> 0.00 mm, vias 3 -> 0
- net /A8: track 0.00 -> 86.2 mm, vias 0 -> 3
- net A9: track 83.8 -> 0.00 mm, vias 2 -> 0
- net /A9: track 0.00 -> 83.8 mm, vias 0 -> 2
- net A10: track 77.4 -> 0.00 mm, vias 1 -> 0
- net /A10: track 0.00 -> 77.4 mm, vias 0 -> 1
- net A15: track 72.0 -> 0.00 mm
- net /A15: track 0.00 -> 72.0 mm
- net A5: track 57.9 -> 0.00 mm
- net /A5: track 0.00 -> 57.9 mm
- net A4: track 57.7 -> 0.00 mm
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Other:
- board outline removed

Commit message: Schematic changes, test script
Parts:
- removed the J2 at (23.6, 115.6)
- removed the R12 at (154.9, 76.2)
- removed the R13 at (154.9, 73.7)
- removed the R15 at (154.9, 68.6)
- removed R17, R19, R20, R21, R22, R23, R24, R25, R26, R27, R28, R29, R30, R31, R32, R33, R34, R35, R36, R39, R40, R41, R47, R49, R50, R51: 1K, Resistor_SMD:R_0603_1608Metric_Pad0.98x0.95mm_HandSolder
- removed R37, R38, R40, R41, R42, R43, R44, R45, R46, R48: 10K, Resistor_SMD:R_0603_1608Metric_Pad0.98x0.95mm_HandSolder
- removed REF**: Symbol_GNU-GPL_SilkscreenFront_Small, Footprints:Symbol_GNU-GPL_SilkscreenFront_Small
- removed SW13, SW14: SW_DIP_x08, Button_Switch_THT:SW_DIP_SPSTx08_Piano_10.8x21.88mm_W7.62mm_P2.54mm
- removed SW5: SW_DIP_x08, Button_Switch_THT:SW_DIP_SPSTx08_Slide_9.78x22.5mm_W7.62mm_P2.54mm
- removed U17, U18, U19, U20, U9: 74LS174, Package_SO:SO-16_5.3x10.2mm_P1.27mm
- removed U20, U23: SST39SF040, Package_DIP:DIP-32_W15.24mm_Socket
- added C8: 1uF, Capacitor_SMD:C_0603_1608Metric, F.Cu at (153.4, 91.9)
- added D2: LED_Blue, LED_SMD:LED_0603_1608Metric, F.Cu at (113.5, 80.3)
- added D21: LED_Red, LED_SMD:LED_0603_1608Metric, F.Cu at (267.2, 54.6)
- added D22: LED_Red, LED_SMD:LED_0603_1608Metric, F.Cu at (271.1, 58.2)
- added D23: LED_Red, LED_SMD:LED_0603_1608Metric, F.Cu at (261.6, 59.7)
- added D24: LED_Red, LED_SMD:LED_0603_1608Metric, F.Cu at (262.9, 64.8)
- added D25: LED_Red, LED_SMD:LED_0603_1608Metric, F.Cu at (268.1, 63.5)
- added D26: LED_Red, LED_SMD:LED_0603_1608Metric, F.Cu at (262.3, 69.8)
- added D27: LED_Red, LED_SMD:LED_0603_1608Metric, F.Cu at (264.8, 95.1)
- added D28: LED_Red, LED_SMD:LED_0603_1608Metric, F.Cu at (267.3, 95.1)
- added D29: LED_Red, LED_SMD:LED_0603_1608Metric, F.Cu at (269.9, 95.1)
- added D30: LED_Red, LED_SMD:LED_0603_1608Metric, F.Cu at (272.4, 95.1)
- added D31: LED_Red, LED_SMD:LED_0603_1608Metric, F.Cu at (275.0, 95.1)
- added D32: LED_Red, LED_SMD:LED_0603_1608Metric, F.Cu at (277.5, 95.1)
- added D33: LED_Red, LED_SMD:LED_0603_1608Metric, F.Cu at (280.0, 95.1)
- added D4: LED_Blue, LED_SMD:LED_0603_1608Metric, F.Cu at (113.5, 85.3)
- added D8: LED_Blue, LED_SMD:LED_0603_1608Metric, F.Cu at (107.4, 84.6)
- added J4: PinHeader_Female04x02, Connector_PinSocket_2.54mm:PinSocket_2x04_P2.54mm_Vertical, F.Cu at (227.3, 52.7)
- added J5: PinHeader_Female04x02, Connector_PinSocket_2.54mm:PinSocket_2x04_P2.54mm_Vertical, F.Cu at (227.3, 66.0)
- added J6: PinHeader_Female04x02, Connector_PinSocket_2.54mm:PinSocket_2x04_P2.54mm_Vertical, F.Cu at (227.3, 79.4)
- added J7: PinHeader_Female04x02, Connector_PinSocket_2.54mm:PinSocket_2x04_P2.54mm_Vertical, F.Cu at (47.4, 121.9)
- added J8: PinHeader_Female04x02, Connector_PinSocket_2.54mm:PinSocket_2x04_P2.54mm_Vertical, F.Cu at (54.6, 121.9)
- added J9: PinHeader_Female04x02, Connector_PinSocket_2.54mm:PinSocket_2x04_P2.54mm_Vertical, F.Cu at (61.7, 121.9)
- added R10: 1K, Resistor_SMD:R_0603_1608Metric, F.Cu at (110.2, 85.3)
- added R3: 1K, Resistor_SMD:R_0603_1608Metric, F.Cu at (110.2, 80.3)
- added R4: 10K, Resistor_SMD:R_0603_1608Metric, B.Cu at (122.6, 85.1)
- added RN1: EXB-D10C102J, r_network:EXB-D10C103J, F.Cu at (291.0, 53.9)
- added RN2: EXB-D10C102J, r_network:EXB-D10C103J, F.Cu at (296.9, 86.8)
- added RN3: EXB-D10C102J, r_network:EXB-D10C103J, F.Cu at (274.6, 66.3)
- added RN4: EXB-D10C102J, r_network:EXB-D10C103J, F.Cu at (271.5, 86.8)
- added RN5: EXB-D10C102J, r_network:EXB-D10C103J, F.Cu at (330.4, 86.7)
- added RN6: EXB-D10C102J, r_network:EXB-D10C103J, F.Cu at (336.2, 86.7)
- added RN7: EXB-D10C102J, r_network:EXB-D10C103J, F.Cu at (56.6, 134.0)
- added RV1: 1M, Potentiometer_SMD:Potentiometer_Vishay_TS53YJ_Vertical, F.Cu at (106.2, 99.8)
- added SW1: SW_Push, Button_Switch_SMD:SW_SPST_B3S-1000, F.Cu at (121.2, 108.0)
- added SW2: SW_SP3T, SP3T_THT:MHS133G04, F.Cu at (98.6, 83.6)
- added SW3: SW_Push, Button_Switch_SMD:SW_SPST_B3S-1000, F.Cu at (153.8, 98.3)
- added U4: SN74HC138N, Package_SO:SOIC-16W_5.3x10.2mm_P1.27mm, F.Cu at (70.6, 25.4)
- added U5: SN74HC138N, Package_SO:SOIC-16W_5.3x10.2mm_P1.27mm, F.Cu at (80.8, 25.4)
- added U6: 4069, Package_SO:SOIC-14_3.9x8.7mm_P1.27mm, F.Cu at (267.2, 71.1)
- added U7: 82C55A, Package_DIP:DIP-40_W15.24mm, F.Cu at (198.8, 52.1)
- added U8: 4081, Package_SO:SO-14_3.9x8.65mm_P1.27mm, F.Cu at (90.1, 24.5)
- C1, C2, C3, C4, C5, C6, C7: footprint Capacitor_SMD:C_0805_2012Metric_Pad1.18x1.45mm_HandSolder -> Capacitor_SMD:C_0603_1608Metric
- CLK1: footprint Package_DIP:DIP-14_W7.62mm_Socket -> Package_SO:SOIC-14_3.9x8.7mm_P1.27mm
- CPU1: value Z84C0010PEG -> Z84C0010AEG; footprint Package_DIP:DIP-40_W15.24mm_Socket -> Package_QFP:LQFP-44_10x10mm_P0.8mm
- D13: renamed from D19; value LED_Small -> LED_Yellow; footprint LED_SMD:LED_0603_1608Metric_Pad1.05x0.95mm_HandSolder -> LED_SMD:LED_0603_1608Metric
- D14: renamed from D20; value LED_Small -> LED_Yellow; footprint LED_SMD:LED_0603_1608Metric_Pad1.05x0.95mm_HandSolder -> LED_SMD:LED_0603_1608Metric
- D15: renamed from D21; value LED_Small -> LED_Yellow; footprint LED_SMD:LED_0603_1608Metric_Pad1.05x0.95mm_HandSolder -> LED_SMD:LED_0603_1608Metric
- D16: renamed from D22; value LED_Small -> LED_Yellow; footprint LED_SMD:LED_0603_1608Metric_Pad1.05x0.95mm_HandSolder -> LED_SMD:LED_0603_1608Metric
- D17: renamed from D23; value LED_Small -> LED_Yellow; footprint LED_SMD:LED_0603_1608Metric_Pad1.05x0.95mm_HandSolder -> LED_SMD:LED_0603_1608Metric
- D18: renamed from D24; value LED_Small -> LED_Yellow; footprint LED_SMD:LED_0603_1608Metric_Pad1.05x0.95mm_HandSolder -> LED_SMD:LED_0603_1608Metric
- D19: renamed from D25; value LED_Small -> LED_Yellow; footprint LED_SMD:LED_0603_1608Metric_Pad1.05x0.95mm_HandSolder -> LED_SMD:LED_0603_1608Metric
- D20: renamed from D26; value LED_Small -> LED_Yellow; footprint LED_SMD:LED_0603_1608Metric_Pad1.05x0.95mm_HandSolder -> LED_SMD:LED_0603_1608Metric
- D34: renamed from D3; value LED_Small -> LED_Yellow; footprint LED_SMD:LED_0603_1608Metric_Pad1.05x0.95mm_HandSolder -> LED_SMD:LED_0603_1608Metric
- D35: renamed from D4; value LED_Small -> LED_Yellow; footprint LED_SMD:LED_0603_1608Metric_Pad1.05x0.95mm_HandSolder -> LED_SMD:LED_0603_1608Metric
- D36: renamed from D5; value LED_Small -> LED_Yellow; footprint LED_SMD:LED_0603_1608Metric_Pad1.05x0.95mm_HandSolder -> LED_SMD:LED_0603_1608Metric
- D37: renamed from D6; value LED_Small -> LED_Yellow; footprint LED_SMD:LED_0603_1608Metric_Pad1.05x0.95mm_HandSolder -> LED_SMD:LED_0603_1608Metric
- D38: renamed from D7; value LED_Small -> LED_Yellow; footprint LED_SMD:LED_0603_1608Metric_Pad1.05x0.95mm_HandSolder -> LED_SMD:LED_0603_1608Metric
- D39: renamed from D8; value LED_Small -> LED_Yellow; footprint LED_SMD:LED_0603_1608Metric_Pad1.05x0.95mm_HandSolder -> LED_SMD:LED_0603_1608Metric
- D40: renamed from D9; value LED_Small -> LED_Yellow; footprint LED_SMD:LED_0603_1608Metric_Pad1.05x0.95mm_HandSolder -> LED_SMD:LED_0603_1608Metric
- D41: renamed from D10; value LED_Small -> LED_Yellow; footprint LED_SMD:LED_0603_1608Metric_Pad1.05x0.95mm_HandSolder -> LED_SMD:LED_0603_1608Metric
- D42: renamed from D11; value LED_Small -> LED_Yellow; footprint LED_SMD:LED_0603_1608Metric_Pad1.05x0.95mm_HandSolder -> LED_SMD:LED_0603_1608Metric
- D43: renamed from D12; value LED_Small -> LED_Yellow; footprint LED_SMD:LED_0603_1608Metric_Pad1.05x0.95mm_HandSolder -> LED_SMD:LED_0603_1608Metric
- D44: renamed from D13; value LED_Small -> LED_Yellow; footprint LED_SMD:LED_0603_1608Metric_Pad1.05x0.95mm_HandSolder -> LED_SMD:LED_0603_1608Metric
- D45: renamed from D14; value LED_Small -> LED_Yellow; footprint LED_SMD:LED_0603_1608Metric_Pad1.05x0.95mm_HandSolder -> LED_SMD:LED_0603_1608Metric
- D46: renamed from D15; value LED_Small -> LED_Yellow; footprint LED_SMD:LED_0603_1608Metric_Pad1.05x0.95mm_HandSolder -> LED_SMD:LED_0603_1608Metric
- D47: renamed from D16; value LED_Small -> LED_Yellow; footprint LED_SMD:LED_0603_1608Metric_Pad1.05x0.95mm_HandSolder -> LED_SMD:LED_0603_1608Metric
- D48: renamed from D17; value LED_Small -> LED_Yellow; footprint LED_SMD:LED_0603_1608Metric_Pad1.05x0.95mm_HandSolder -> LED_SMD:LED_0603_1608Metric
- D49: renamed from D18; value LED_Small -> LED_Yellow; footprint LED_SMD:LED_0603_1608Metric_Pad1.05x0.95mm_HandSolder -> LED_SMD:LED_0603_1608Metric
- D5: renamed from D1; value LED -> LED_Blue; footprint LED_SMD:LED_0603_1608Metric_Pad1.05x0.95mm_HandSolder -> LED_SMD:LED_0603_1608Metric
- D6: renamed from D2; value LED -> LED_Blue; footprint LED_SMD:LED_0603_1608Metric_Pad1.05x0.95mm_HandSolder -> LED_SMD:LED_0603_1608Metric
- J1: value Screw_Terminal_01x02 -> PinHeader_Female01x02; footprint TerminalBlock_4Ucon:TerminalBlock_4Ucon_1x02_P3.50mm_Horizontal -> Connector_PinHeader_2.54mm:PinHeader_1x02_P2.54mm_Vertical
- J2: value Conn_02x16_Counter_Clockwise -> PinHeader_Female16x02; footprint Connector_PinSocket_2.54mm:PinSocket_2x16_P2.54mm_Vertical -> Card_Connector:FX2740S08SV
- J3: value Conn_02x16_Counter_Clockwise -> PinHeader_Female16x02; footprint Connector_PinHeader_2.54mm:PinHeader_2x16_P2.54mm_Horizontal -> Card_Connector:FX2740S08SV
- R1, R14, R2: footprint Resistor_SMD:R_0603_1608Metric_Pad0.98x0.95mm_HandSolder -> Resistor_SMD:R_0603_1608Metric
- R11: renamed from R8; footprint Resistor_SMD:R_0603_1608Metric_Pad0.98x0.95mm_HandSolder -> Resistor_SMD:R_0603_1608Metric
- R12: renamed from R9; footprint Resistor_SMD:R_0603_1608Metric_Pad0.98x0.95mm_HandSolder -> Resistor_SMD:R_0603_1608Metric
- R13: renamed from R10; footprint Resistor_SMD:R_0603_1608Metric_Pad0.98x0.95mm_HandSolder -> Resistor_SMD:R_0603_1608Metric
- R15: renamed from R11; footprint Resistor_SMD:R_0603_1608Metric_Pad0.98x0.95mm_HandSolder -> Resistor_SMD:R_0603_1608Metric
- R16, R18: value 1K -> 10K; footprint Resistor_SMD:R_0603_1608Metric_Pad0.98x0.95mm_HandSolder -> Resistor_SMD:R_0603_1608Metric
- R6: renamed from R4; footprint Resistor_SMD:R_0603_1608Metric_Pad0.98x0.95mm_HandSolder -> Resistor_SMD:R_0603_1608Metric
- R7: renamed from R5; footprint Resistor_SMD:R_0603_1608Metric_Pad0.98x0.95mm_HandSolder -> Resistor_SMD:R_0603_1608Metric
- R8: renamed from R6; footprint Resistor_SMD:R_0603_1608Metric_Pad0.98x0.95mm_HandSolder -> Resistor_SMD:R_0603_1608Metric
- R9: renamed from R7; footprint Resistor_SMD:R_0603_1608Metric_Pad0.98x0.95mm_HandSolder -> Resistor_SMD:R_0603_1608Metric
- ROM1: footprint Package_DIP:DIP-28_W15.24mm_Socket -> Package_SO:SOIC-28W_7.5x17.9mm_P1.27mm
- U10: value 74LS174 -> 82C55A; footprint Package_SO:SO-16_5.3x10.2mm_P1.27mm -> Package_DIP:DIP-40_W15.24mm
- moved J3 207.1 mm to (184.6, 75.2), turned to -90 degrees
- moved D49 195.2 mm to (352.4, 95.1), turned to 90 degrees
- moved D48 192.0 mm to (349.9, 95.1), turned to 90 degrees
- moved J1 189.0 mm to (226.1, 92.7)
- moved D47 188.7 mm to (347.3, 95.1), turned to 90 degrees
- moved D46 185.5 mm to (344.8, 95.1), turned to 90 degrees
- moved D41 184.6 mm to (332.1, 95.1), turned to 90 degrees
- moved D45 182.3 mm to (342.3, 95.1), turned to 90 degrees
- moved D40 181.7 mm to (329.6, 95.1), turned to 90 degrees
- moved D44 179.1 mm to (339.7, 95.1), turned to 90 degrees
- moved D39 178.7 mm to (327.0, 95.1), turned to 90 degrees
- moved D43 175.9 mm to (337.2, 95.1), turned to 90 degrees
- moved D38 175.8 mm to (324.5, 95.1), turned to 90 degrees
- moved D37 172.9 mm to (321.9, 95.1), turned to 90 degrees
- moved D42 172.8 mm to (334.6, 95.1), turned to 90 degrees
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- renumbered X8.000Mhz1 to CLK2, R3 to R5
Connections:
- A1 pad 10: unconnected-(A1-Pad10) -> Net-(A1-D14)
- A1 pad 11: unconnected-(A1-Pad11) -> Net-(A1-D16)
- A1 pad 12: unconnected-(A1-Pad12) -> /BUSRQ
- A1 pad 13: unconnected-(A1-Pad13) -> /D7
- A1 pad 14: unconnected-(A1-Pad14) -> /D6
- A1 pad 15: unconnected-(A1-Pad15) -> /D5
- A1 pad 16: unconnected-(A1-Pad16) -> /D4
- A1 pad 17: unconnected-(A1-Pad17) -> /D3
- A1 pad 18: unconnected-(A1-Pad18) -> /D2
- A1 pad 19: unconnected-(A1-Pad19) -> /D1
- A1 pad 2: unconnected-(A1-Pad2) -> GND
- A1 pad 20: unconnected-(A1-Pad20) -> /D0
- A1 pad 21: unconnected-(A1-Pad21) -> GND
- A1 pad 22: unconnected-(A1-Pad22) -> GND
- A1 pad 4: unconnected-(A1-Pad4) -> +5V
- A1 pad 5: unconnected-(A1-Pad5) -> /BUSACK
- A1 pad 6: Net-(A1-Pad6) -> Net-(A1-A2)
- A1 pad 7: unconnected-(A1-Pad7) -> /PROG-WR
- A1 pad 8: unconnected-(A1-Pad8) -> /RD
- A1 pad 9: Net-(A1-Pad9) -> Net-(A1-D15)
- CPU1 pad 1: /A11 -> Clock
- CPU1 pad 10: D6 -> /D1
- CPU1 pad 11: +5V -> unconnected-(CPU1-NC-Pad11)
- CPU1 pad 12: D2 -> /INT
- CPU1 pad 13: D7 -> /NMI
- CPU1 pad 14: D0 -> /HALT
- CPU1 pad 15: D1 -> /MREQ
- CPU1 pad 16: /INT -> /IORQ
- CPU1 pad 17: /NMI -> unconnected-(CPU1-NC-Pad17)
- CPU1 pad 18: /HALT -> /RD
- CPU1 pad 19: /MREQ -> /WR
- CPU1 pad 2: /A12 -> /D4
- CPU1 pad 20: /IORQ -> /BUSACK
- CPU1 pad 21: /RD -> /WAIT
- CPU1 pad 22: /WR -> /BUSRQ
- CPU1 pad 23: unconnected-(CPU1-Pad23) -> /RST
- CPU1 pad 24: /WAIT -> /M1
- CPU1 pad 25: unconnected-(CPU1-Pad25) -> /RFSH
- CPU1 pad 26: Net-(CPU1-Pad26) -> GND
- CPU1 pad 27: /M1 -> /A0
- CPU1 pad 28: /RFSH -> /A1
- CPU1 pad 29: GND -> /A2
- CPU1 pad 3: /A13 -> /D3
- CPU1 pad 30: A0 -> /A3
- CPU1 pad 31: A1 -> /A4
- CPU1 pad 32: A2 -> /A5
- CPU1 pad 33: A3 -> unconnected-(CPU1-NC-Pad33)
- CPU1 pad 34: /A4 -> /A6
- CPU1 pad 35: /A5 -> /A7
- CPU1 pad 36: /A6 -> /A8
- CPU1 pad 37: /A7 -> /A9
- CPU1 pad 38: /A8 -> /A10
- CPU1 pad 39: /A9 -> unconnected-(CPU1-NC-Pad39)
- CPU1 pad 4: /A14 -> /D5
- CPU1 pad 40: /A10 -> /A11
- CPU1 pad 5: /A15 -> /D6
- CPU1 pad 6: Clock -> +5V
- CPU1 pad 7: D4 -> /D2
- CPU1 pad 8: D3 -> /D7
- CPU1 pad 9: D5 -> /D0
- D13 pad 2: D0 -> /D0
- D14 pad 2: D1 -> /D1
- D15 pad 2: D2 -> /D2
- D16 pad 2: D3 -> /D3
- D17 pad 2: D4 -> /D4
- D18 pad 2: D5 -> /D5
- D19 pad 2: D6 -> /D6
- D20 pad 2: D7 -> /D7
- D34 pad 2: A0 -> /A0
- D35 pad 2: A1 -> /A1
- D36 pad 1: Net-(D5-Pad1) -> Net-(D36-K)
- D36 pad 2: A2 -> /A2
- D37 pad 2: A3 -> /A3
- D38 pad 1: Net-(D7-Pad1) -> Net-(D38-K)
- D40 pad 1: Net-(D9-Pad1) -> Net-(D40-K)
- J2 pad 1: D7 -> /D7
- J2 pad 10: +5V -> /IORQ
- J2 pad 11: /RST -> /MREQ
- J2 pad 12: /IORQ -> /RD
- J2 pad 13: /MREQ -> /WR
- J2 pad 14: /RD -> /INT
- J2 pad 15: /WR -> /NMI
- J2 pad 16: GND -> /WAIT
- J2 pad 17: GND -> /EXT-IO2-CS
- J2 pad 18: A0 -> /EXT-IO1-CS
- J2 pad 19: A1 -> +5V
- J2 pad 2: D6 -> /D6
- J2 pad 20: A2 -> +5V
- J2 pad 21: A3 -> /A15
- J2 pad 22: /A4 -> /A14
- J2 pad 23: /A5 -> /A13
- J2 pad 24: /A6 -> /A12
- J2 pad 25: /A7 -> /A11
- J2 pad 26: /A8 -> /A10
- J2 pad 28: /A10 -> /A8
- J2 pad 29: /A11 -> /A7
- J2 pad 3: D5 -> /D5
- J2 pad 30: /A12 -> /A6
- J2 pad 31: /A13 -> /A5
- J2 pad 32: /A14 -> /A4
- J2 pad 4: D4 -> /D4
- J2 pad 5: D3 -> /D3
- J2 pad 6: D2 -> /D2
- J2 pad 7: D1 -> /D1
- J2 pad 8: D0 -> /D0
- J2 pad 9: /A15 -> /RST
- J3 pad 1: /Flash Cartridge/D7 -> /D7
- J3 pad 10: /Flash Cartridge/PWR -> /IORQ
- J3 pad 11: /Flash Cartridge/RST -> /MREQ
- J3 pad 12: /Flash Cartridge/IO -> /RD
- J3 pad 13: /Flash Cartridge/MEM -> /WR
- J3 pad 14: /Flash Cartridge/RD -> /INT
- J3 pad 15: /Flash Cartridge/WR -> /NMI
- J3 pad 16: Net-(J3-Pad16) -> /WAIT
- J3 pad 17: Net-(J3-Pad16) -> /EXT-IO5-CS
- J3 pad 18: /Flash Cartridge/A0 -> /EXT-IO4-CS
- J3 pad 19: /Flash Cartridge/A1 -> +5V
- J3 pad 2: /Flash Cartridge/D6 -> /D6
- J3 pad 20: /Flash Cartridge/A2 -> +5V
- J3 pad 21: /Flash Cartridge/A3 -> /A15
- J3 pad 22: /Flash Cartridge/A4 -> /A14
- J3 pad 23: /Flash Cartridge/A5 -> /A13
- J3 pad 24: /Flash Cartridge/A6 -> /A12
- J3 pad 25: /Flash Cartridge/A7 -> /A11
- J3 pad 26: /Flash Cartridge/A8 -> /A10
- J3 pad 27: /Flash Cartridge/A9 -> /A9
- J3 pad 28: /Flash Cartridge/A10 -> /A8
- J3 pad 29: /Flash Cartridge/A11 -> /A7
- J3 pad 3: /Flash Cartridge/D5 -> /D5
- J3 pad 30: /Flash Cartridge/A12 -> /A6
- J3 pad 31: /Flash Cartridge/A13 -> /A5
- J3 pad 32: /Flash Cartridge/A14 -> /A4
- J3 pad 4: /Flash Cartridge/D4 -> /D4
- J3 pad 5: /Flash Cartridge/D3 -> /D3
- J3 pad 6: /Flash Cartridge/D2 -> /D2
- J3 pad 7: /Flash Cartridge/D1 -> /D1
- J3 pad 8: /Flash Cartridge/D0 -> /D0
- J3 pad 9: /Flash Cartridge/A15 -> /RST
- R14 pad 1: GND -> Net-(D8-K)
- R14 pad 2: Net-(D5-Pad1) -> GND
- R15 pad 2: Net-(CPU1-Pad26) -> +5V
- R16 pad 1: GND -> +5V
- R16 pad 2: Net-(D7-Pad1) -> /PROG-WR
- R18 pad 1: GND -> /RST-INV
- R18 pad 2: Net-(D9-Pad1) -> +5V
- RAM1 pad 10: A0 -> /A0
- RAM1 pad 11: D0 -> /D0
- RAM1 pad 12: D1 -> /D1
- RAM1 pad 13: D2 -> /D2
- RAM1 pad 15: D3 -> /D3
- RAM1 pad 16: D4 -> /D4
- RAM1 pad 17: D5 -> /D5
- RAM1 pad 18: D6 -> /D6
- RAM1 pad 19: D7 -> /D7
- RAM1 pad 7: A3 -> /A3
- RAM1 pad 8: A2 -> /A2
- RAM1 pad 9: A1 -> /A1
- ROM1 pad 10: A0 -> /A0
- ROM1 pad 11: D0 -> /D0
- ROM1 pad 12: D1 -> /D1
- ROM1 pad 13: D2 -> /D2
- ROM1 pad 15: D3 -> /D3
- ROM1 pad 16: D4 -> /D4
- ROM1 pad 17: D5 -> /D5
- ROM1 pad 18: D6 -> /D6
- ROM1 pad 19: D7 -> /D7
- ROM1 pad 27: /WR -> /PROG-WR
- ROM1 pad 7: A3 -> /A3
- ROM1 pad 8: A2 -> /A2
- ROM1 pad 9: A1 -> /A1
- U1 pad 10: Clock -> Net-(D7-A)
- U1 pad 11: (no net) -> /ROM1-CS
- U1 pad 12: (no net) -> Net-(U4-Y1)
- U1 pad 13: (no net) -> Net-(U4-Y0)
- U1 pad 3: Clock -> Net-(D1-A)
- U1 pad 4: Clock -> Net-(D3-A)
- U10 pad 10: unconnected-(U10-Pad10) -> Net-(J9-Pin_7)
- U10 pad 11: unconnected-(U10-Pad11) -> Net-(J9-Pin_5)
- U10 pad 12: unconnected-(U10-Pad12) -> Net-(J9-Pin_3)
- U10 pad 13: unconnected-(U10-Pad13) -> Net-(J9-Pin_1)
- U10 pad 14: unconnected-(U10-Pad14) -> Net-(J9-Pin_2)
- U10 pad 15: unconnected-(U10-Pad15) -> Net-(J9-Pin_4)
- U10 pad 16: +5V -> Net-(J9-Pin_6)
- U10 pad 2: /Clk -> Net-(J7-Pin_6)
- U10 pad 4: unconnected-(U10-Pad4) -> Net-(J7-Pin_2)
- U10 pad 5: unconnected-(U10-Pad5) -> /RD
- U10 pad 6: unconnected-(U10-Pad6) -> /IO2-CS
- U10 pad 7: unconnected-(U10-Pad7) -> GND
- U10 pad 8: GND -> /A1
- U10 pad 9: Net-(U7-Pad4) -> /A0
- U2 pad 1: A1 -> /A1
- U2 pad 11: Net-(A1-Pad27) -> Net-(A1-D14)
- U2 pad 12: Net-(A1-Pad26) -> Net-(A1-D16)
- U2 pad 13: GND -> Net-(A1-A2)
- U2 pad 14: Net-(A1-Pad28) -> Net-(A1-D15)
- U2 pad 15: A0 -> /A0
- U2 pad 2: A2 -> /A2
- U2 pad 3: A3 -> /A3
- U3 pad 11: Net-(A1-Pad27) -> Net-(A1-D14)
- U3 pad 12: Net-(A1-Pad26) -> Net-(A1-D16)
- U3 pad 13: GND -> Net-(A1-A2)
Routing:
- net /A11: track 95.9 -> 0.00 mm, vias 2 -> 0
- net /A12: track 90.0 -> 0.00 mm, vias 1 -> 0
- net D6: track 88.5 -> 0.00 mm, vias 3 -> 0
- net /MREQ: track 88.4 -> 0.00 mm
- net /A8: track 86.2 -> 0.00 mm, vias 3 -> 0
- net /A9: track 83.8 -> 0.00 mm, vias 2 -> 0
- net D4: track 82.7 -> 0.00 mm, vias 2 -> 0
- net D5: track 81.8 -> 0.00 mm, vias 4 -> 0
- net /A10: track 77.4 -> 0.00 mm, vias 1 -> 0
- net /D4: track 0.00 -> 76.5 mm, vias 0 -> 4
- net /IORQ: track 75.5 -> 0.00 mm, vias 1 -> 0
- net /D3: track 0.00 -> 74.7 mm, vias 0 -> 4
- net /D0: track 0.00 -> 74.5 mm, vias 0 -> 2
- net D3: track 74.4 -> 0.00 mm
- net D7: track 74.2 -> 0.00 mm, vias 2 -> 0
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Other:
- copper layers 2 -> 4
- board text added: "+5V"
- board text added: "0"
- board text added: "15"
- board text added: "7"
- board text added: "Address"
- board text added: "B0"
- board text added: "B1"
- board text added: "B2"
- board text added: "B3"
- board text added: "B4"
- board text added: "B5"
- board text added: "B6"
- board text added: "B7"
- board text added: "Bus Ack"
- board text added: "Bus Req"
- board text added: "C0"
- board text added: "C1"
- board text added: "C2"
- board text added: "C3"
- board text added: "C4"
- board text added: "C5"
- board text added: "C6"
- board text added: "C7"
- board text added: "Control"
- board text added: "Data"
- board text added: "GND"
- board text added: "IO"
- board text added: "IO Req"
- board text added: "Mem Req"
- board text added: "Oscillator"
- board text added: "PWR"
- board text added: "Read"
- board text added: "Reset"
- board text added: "Timer"
- board text added: "Write"
- board text removed: "A10"
- board text removed: "A11"
- board text removed: "A12"
- board text removed: "A13"
- board text removed: "A14"
- board text removed: "A15"
- board text removed: "A8"
- board text removed: "A9"
- board text removed: "D0"
- board text removed: "D1"
- board text removed: "D2"
- board text removed: "D3"
- board text removed: "D4"
- board text removed: "D5"
- board text removed: "D6"
- board text removed: "D7"

Commit message: Schematic cahnges, PCB changes, test asm changes
Parts:
- RN7: moved to B.Cu
- moved RN7 102.7 mm to (140.8, 75.3)
- moved U3 95.1 mm to (145.0, 42.9)
- moved U2 91.8 mm to (131.6, 42.9)
- moved R16 71.9 mm to (141.5, 57.9), turned to -90 degrees
- moved RAM1 27.3 mm to (173.5, -4.06)
- moved J6 17.8 mm to (226.0, 61.6)
- moved J4 17.8 mm to (225.9, 34.9)
- moved U7 17.8 mm to (197.4, 34.3)
- moved J5 17.8 mm to (226.0, 48.3)
- moved R18 17.8 mm to (215.6, 47.0)
- moved J1 17.8 mm to (224.7, 74.9)
- moved R15 9.22 mm to (147.3, 96.8), turned to -90 degrees
- moved C8 8.39 mm to (160.3, 96.8), turned to 90 degrees
- moved J2 6.02 mm to (164.5, 73.0)
- moved J3 6.02 mm to (179.0, 73.0)
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Routing:
- net /A1: track 0.00 -> 176.1 mm, vias 0 -> 4
- net /A2: track 0.00 -> 166.9 mm, vias 0 -> 4
- net /A0: track 0.00 -> 158.9 mm, vias 0 -> 2
- net /A3: track 0.00 -> 148.1 mm, vias 0 -> 4
- net /A4: track 0.00 -> 140.1 mm, vias 0 -> 4
- net /A5: track 0.00 -> 132.0 mm, vias 0 -> 2
- net /A6: track 0.00 -> 124.4 mm, vias 0 -> 4
- net /A7: track 0.00 -> 119.1 mm, vias 0 -> 4
- net +5V: track 149.3 -> 32.7 mm, vias 1 -> 16
- net /A12: track 0.00 -> 109.4 mm, vias 0 -> 5
- net /A9: track 0.00 -> 108.8 mm, vias 0 -> 4
- net /A8: track 0.00 -> 108.1 mm, vias 0 -> 4
- net /A10: track 0.00 -> 106.7 mm, vias 0 -> 4
- net /A11: track 0.00 -> 101.8 mm, vias 0 -> 5
- net /BUSACK: track 0.00 -> 65.2 mm, vias 0 -> 1
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Other:
- board text added: "z80 Main Board Rev.1 Designed by Tristan van de Weg & Marijn Vollenberg"
- board text removed: "z80 Main Board Designed by Tristan van de Weg & Marijn Vollenberg"

Commit message: Board revision 1
Parts:
- added REF**: MountingHole_3.2mm_M3, MountingHole:MountingHole_3.2mm_M3, F.Cu at (92.4, 33.9)
- added REF**: MountingHole_3.2mm_M3, MountingHole:MountingHole_3.2mm_M3, F.Cu at (229.6, 135.9)
- added REF**: MountingHole_3.2mm_M3, MountingHole:MountingHole_3.2mm_M3, F.Cu at (119.3, 135.8)
- added REF**: MountingHole_3.2mm_M3, MountingHole:MountingHole_3.2mm_M3, F.Cu at (188.1, 33.9)
- added U9: 74LS32, Package_SO:SOIC-14_3.9x8.7mm_P1.27mm, F.Cu at (134.6, 95.2)
- C8: footprint Capacitor_SMD:C_0603_1608Metric -> Capacitor_SMD:C_1206_3216Metric
- RAM1: footprint Package_DIP:DIP-28_W15.24mm_Socket -> Package_SO:TSOP-I-28_11.8x8mm_P0.55mm
- RN2, RN3, RN4, RN5, RN6: moved to B.Cu
- moved D22 189.4 mm to (91.6, 118.3), turned to 90 degrees
- moved D21 189.2 mm to (89.0, 118.3), turned to 90 degrees
- moved RN3 187.9 mm to (94.1, 118.3), turned to -90 degrees
- moved J7 181.2 mm to (225.9, 90.9)
- moved D25 177.6 mm to (99.2, 118.3), turned to 90 degrees
- moved D23 177.5 mm to (94.1, 118.3), turned to 90 degrees
- moved D24 174.7 mm to (96.6, 118.3), turned to 90 degrees
- moved U10 174.5 mm to (197.4, 90.2)
- moved J8 172.3 mm to (226.0, 104.2)
- moved RN5 170.8 mm to (162.6, 118.0)
- moved D26 167.7 mm to (101.7, 118.3), turned to 90 degrees
- moved J9 164.3 mm to (226.0, 117.6)
- moved RN2 163.6 mm to (136.4, 118.3)
- moved RN4 162.7 mm to (111.9, 118.3), turned to -90 degrees
- moved D13 162.2 mm to (127.8, 118.3)
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Connections:
- A1 pad 6: Net-(A1-A2) -> /PROG-OE
- R18 pad 2: +5V -> GND
- RN1 pad 6: /IORQ -> unconnected-(RN1-R5-Pad6)
- U1 pad 10: Net-(D7-A) -> /ManOUT
- U1 pad 11: /ROM1-CS -> /EXT-CS
- U1 pad 12: Net-(U4-Y1) -> Net-(U1-Pad12)
- U1 pad 13: Net-(U4-Y0) -> Net-(U1-Pad13)
- U1 pad 3: Net-(D1-A) -> /FstOUT
- U1 pad 4: Net-(D3-A) -> /AdjOUT
- U2 pad 13: Net-(A1-A2) -> /PROG-OE
- U3 pad 13: Net-(A1-A2) -> /PROG-OE
- U4 pad 14: Net-(U4-Y1) -> /RAM1-CS
- U4 pad 15: Net-(U4-Y0) -> /ROM1-CS
- U4 pad 6: /IORQ -> /IOREQ
- U5 pad 4: /IORQ -> /IOREQ
- U6 pad 3: unconnected-(U6-Pad3) -> /PROG-OE
- U6 pad 4: unconnected-(U6-Pad4) -> Net-(U6-Pad4)
- U8 pad 11: /RAM1-CS -> Net-(U1-Pad13)
- U8 pad 3: /EXT-CS -> Net-(U1-Pad12)
Routing:
- net /WR: track 0.00 -> 435.9 mm, vias 0 -> 12
- net /RD: track 26.8 -> 313.5 mm, vias 1 -> 10
- net /D3: track 36.9 -> 306.0 mm, vias 4 -> 9
- net /D2: track 88.7 -> 310.1 mm, vias 5 -> 10
- net /D7: track 89.3 -> 310.6 mm, vias 5 -> 11
- net /D6: track 92.1 -> 305.2 mm, vias 7 -> 12
- net /D5: track 90.7 -> 303.3 mm, vias 7 -> 13
- net /D0: track 93.3 -> 303.4 mm, vias 5 -> 9
- net /D4: track 81.2 -> 287.6 mm, vias 6 -> 10
- net /D1: track 91.8 -> 297.7 mm, vias 5 -> 10
- net /MREQ: track 0.00 -> 179.8 mm, vias 0 -> 9
- net /WAIT: track 0.00 -> 145.6 mm, vias 0 -> 5
- net /A13: track 38.7 -> 181.6 mm, vias 3 -> 9
- net /A14: track 40.6 -> 181.7 mm, vias 3 -> 8
- net /NMI: track 0.00 -> 140.4 mm, vias 0 -> 7
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- added copper zone on In2.Cu, net +5V
- added copper zone on B.Cu, net GND
- added copper zone on F.Cu, net GND
- added copper zone on In1.Cu, net GND
Other:
- board outline added: 149.2 x 113.9 mm
- board text added: "Bus Acknowledge"
- board text added: "Bus Request"
- board text added: "Halt"
- board text added: "IO 1"
- board text added: "IO 2"
- board text added: "IO Request"
- board text added: "Interrupt"
- board text added: "Machine Cycle One"
- board text added: "Manual"
- board text added: "Memory Request"
- board text added: "Non-Maskable Interrupt"
- board text added: "Refresh"
- board text added: "Wait"
- board text removed: "Bus Ack"
- board text removed: "Bus Req"
- board text removed: "IO"
- board text removed: "IO Req"
- board text removed: "Mem Req"

Commit message: Schematic/code changes, updated to 2024
Parts:
- added C10: 22pF, Capacitor_SMD:C_0603_1608Metric, F.Cu at (43.1, 67.1)
- added C11: 1uF, Capacitor_SMD:C_0603_1608Metric, F.Cu at (43.1, 69.6)
- added C12: 1uF, Capacitor_SMD:C_0603_1608Metric, F.Cu at (43.1, 72.1)
- added C9: 22pF, Capacitor_SMD:C_0603_1608Metric, F.Cu at (43.1, 64.6)
- added D1: Red, LED_SMD:LED_0603_1608Metric, F.Cu at (61.6, 64.7)
- added J10: Conn_02x03_Counter_Clockwise, Connector_PinHeader_2.54mm:PinHeader_2x03_P2.54mm_Vertical, F.Cu at (59.1, 80.1)
- added J11: USB_C_Receptacle_USB2.0, Connector_USB:USB_C_Receptacle_Palconn_UTC16-G, F.Cu at (50.9, 81.9)
- added R17: 22R, Resistor_SMD:R_0603_1608Metric, F.Cu at (43.1, 77.2)
- added R19: 22R, Resistor_SMD:R_0603_1608Metric, F.Cu at (43.1, 79.7)
- added R20: 10K, Resistor_SMD:R_0603_1608Metric, F.Cu at (43.1, 82.2)
- added R21: 1K, Resistor_SMD:R_0603_1608Metric, F.Cu at (43.1, 84.7)
- added R4: 10K, Resistor_SMD:R_0603_1608Metric, F.Cu at (43.1, 74.7)
- added U11: ATmega32U4RC-A, Package_QFP:TQFP-44_10x10mm_P0.8mm, F.Cu at (52.4, 70.6)
- C1: footprint Capacitor_SMD:C_0603_1608Metric -> Capacitor_SMD:C_1206_3216Metric
- C8: footprint Capacitor_SMD:C_1206_3216Metric -> Capacitor_SMD:C_0603_1608Metric
Connections:
- SW2 pad 1: Net-(R8-Pad2) -> Net-(D2-A)
- SW2 pad 2: Net-(D2-A) -> Net-(R8-Pad2)
Routing:
- net GND: track 100.0 -> 93.8 mm, vias 48 -> 45
- net /D7: track 310.6 -> 313.1 mm, vias 11 -> 12
- net +5V: track 101.2 -> 99.3 mm, vias 26 -> 25
- net /A10: track 204.2 -> 206.1 mm, vias 9 -> 10
- net /RD: track 313.5 -> 315.3 mm, vias 10 -> 11
- net /A3: track 224.3 -> 226.2 mm, vias 9 -> 10
