File: z80/Peripherals/IO_LED_Stick/IO_LED_Stick.kicad_pcb (KiCad board)
At the start: 2 copper layers, 17.5 x 16.9 mm, 11 parts, among them J1 Conn_02x04_Counter_Clockwise, J2 Conn_01x01

Commit message: finished v2 of hardware, updated eeprom prog pins
Routing:
- net GND: track 0.00 -> 3.52 mm
Changed lines of the file:
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@@
   (segment (start 145.792266 83.824734) (end 147.125 82.492) (width 0.25) (layer "B.Cu") (net 16))
   (segment (start 143.379514 83.824734) (end 145.792266 83.824734) (width 0.25) (layer "B.Cu") (net 16))
+  (segment (start 151.13 84.601401) (end 151.13 88.118599) (width 0.25) (layer "B.Cu") (net 17))
   (zone (net 17) (net_name "GND") (layers "F&B.Cu") (hatch edge 0.5)
-    (connect_pads yes (clearance 0.5))
+    (connect_pads (clearance 0.5))
     (min_thickness 0.25) (filled_areas_thickness no)
-    (fill yes (thermal_gap 0.5) (thermal_bridge_width 0.5))
+    (fill yes (thermal_gap 0.5) (thermal_bridge_width 0.5) (island_removal_mode 2) (island_area_min 10))
     (polygon
       (pts
