File: z80/Peripherals/ROM_Card/ROM_Card.kicad_sch (KiCad schematic)
At the start: 14 parts, among them J1 Conn_02x20_Top_Bottom, SW1 SW_SPDT, SW2 SW_SPDT, SW3 SW_SPDT, SW4 SW_SPDT, SW5 SW_SPDT, SW6 SW_SPDT, SW7 SW_SPDT, SW8 SW_SPDT, U1 74HC244, U2 SST39SF040, U3 74LS174, U4 SN74LVC1G14DBV, U5 74AHC1G02

Commit message: schematic updates, assembly progress
Parts:
- removed U4: SN74LVC1G14DBV, Package_TO_SOT_SMD:SOT-23-5, symbol 74xGxx:SN74LVC1G14DBV
- added SW10, SW9: SW_SPDT, Jumper:SolderJumper-3_P1.3mm_Open_Pad1.0x1.5mm, symbol Switch:SW_SPDT
- U1: footprint (none) -> Package_SO:TSSOP-20_4.4x6.5mm_P0.65mm
- U2: footprint (none) -> Package_SO:TSOP-I-32_14.4x8mm_P0.5mm
- U5: footprint (none) -> Package_TO_SOT_SMD:SOT-553
Connections:
- net +5V: no longer J1.19 (Pin_19), U2.31 (PGM)
- net A14: now also SW10.3 (C); no longer U2.29 (A14)
- net A15: no longer U2.3 (A15)
- net A16: now also U2.2 (A16), U3.7 (Q2); no longer U3.2 (Q0)
- net A17: now also U2.30 (A17), U3.10 (Q3); no longer U3.5 (Q1)
- net A18: now also U2.1 (A18), U3.12 (Q4); no longer U3.7 (Q2)
- net CS: now also SW9.3 (C); no longer U2.22 (CE)
- net GND: no longer J1.39 (Pin_39)
- net at U5.4: now also U3.9 (Cp)
- new net: SW9.2 (B), U2.22 (CE)
- new net: SW10.2 (B), U2.29 (A14)
- new net A14B: SW10.1 (A), U3.2 (Q0)
- new net A15B: U2.3 (A15), U3.5 (Q1)
- new net EXT-CS2: J1.39 (Pin_39), SW9.1 (A)
- new net PGM/5V: J1.19 (Pin_19), U2.31 (PGM)
- no-connect marks 0 -> 1
Other:
- moved on the sheet: U5

Commit message: finished v2 of hardware, updated eeprom prog pins
Parts:
- U2: footprint Package_SO:TSOP-I-32_14.4x8mm_P0.5mm -> Package_LCC:PLCC-32_THT-Socket
- U3: footprint (none) -> Package_SO:TSSOP-16_4.4x5mm_P0.65mm
- renumbered SW1 to ID0, SW2 to ID1, SW3 to ID2, SW4 to ID3, SW5 to ID4, SW6 to ID5, SW7 to ID6, SW8 to ID7, SW10 to SA14, SW9 to SCS1
Other:
- title: (none) -> z80 ROM Card
Changed lines of the file:
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@@
 (kicad_sch (version 20230121) (generator eeschema)
   (paper "A4")
+  (title_block
+    (title "z80 ROM Card")
+    (date "2024-03-07")
+    (rev "1.0")
+  )
   (no_connect (at 146.05 31.75))
   (wire (pts (xy 110.49 95.25) (xy 110.49 77.47))
@@
   (symbol (lib_id "Switch:SW_SPDT") (at 101.6 77.47 180) (unit 1)
     (in_bom yes) (on_board yes) (dnp no)
-    (property "Reference" "SW1" (at 100.33 77.47 0)
+    (property "Reference" "ID0" (at 100.33 77.47 0)
       (effects (font (size 1.27 1.27)))
     )
@@
       (project "ROM_Card"
         (path "/5ffe5182-cc98-4b6a-b75c-eae8ba1b784e"
-          (reference "SW1") (unit 1)
+          (reference "ID0") (unit 1)
         )
       )
@@
   (symbol (lib_id "Switch:SW_SPDT") (at 101.6 130.81 180) (unit 1)
     (in_bom yes) (on_board yes) (dnp no)
-    (property "Reference" "SW8" (at 100.33 130.81 0)
+    (property "Reference" "ID7" (at 100.33 130.81 0)
       (effects (font (size 1.27 1.27)))
     )
@@
       (project "ROM_Card"
         (path "/5ffe5182-cc98-4b6a-b75c-eae8ba1b784e"
-          (reference "SW8") (unit 1)
+          (reference "ID7") (unit 1)
         )
       )
@@
   (symbol (lib_id "Switch:SW_SPDT") (at 184.785 86.36 180) (unit 1)
     (in_bom yes) (on_board yes) (dnp no)
-    (property "Reference" "SW9" (at 183.515 86.36 0)
+    (property "Reference" "SCS1" (at 183.515 86.36 0)
       (effects (font (size 1.27 1.27)))
     )
@@
       (project "ROM_Card"
         (path "/5ffe5182-cc98-4b6a-b75c-eae8ba1b784e"
-          (reference "SW9") (unit 1)
+          (reference "SCS1") (unit 1)
         )
       )
@@
       (effects (font (size 1.27 1.27)) (justify left))
     )
-    (property "Footprint" "Package_SO:TSOP-I-32_14.4x8mm_P0.5mm" (at 208.28 53.34 0)
+    (property "Footprint" "Package_LCC:PLCC-32_THT-Socket" (at 208.28 53.34 0)
       (effects (font (size 1.27 1.27)) hide)
     )
@@
   (symbol (lib_id "Switch:SW_SPDT") (at 101.6 115.57 180) (unit 1)
     (in_bom yes) (on_board yes) (dnp no)
-    (property "Reference" "SW6" (at 100.33 115.57 0)
+    (property "Reference" "ID5" (at 100.33 115.57 0)
       (effects (font (size 1.27 1.27)))
     )
@@
       (project "ROM_Card"
         (path "/5ffe5182-cc98-4b6a-b75c-eae8ba1b784e"
-          (reference "SW6") (unit 1)
+          (reference "ID5") (unit 1)
         )
       )
@@
   (symbol (lib_id "Switch:SW_SPDT") (at 101.6 85.09 180) (unit 1)
     (in_bom yes) (on_board yes) (dnp no)
-    (property "Reference" "SW2" (at 100.33 85.09 0)
+    (property "Reference" "ID1" (at 100.33 85.09 0)
       (effects (font (size 1.27 1.27)))
     )
@@
       (project "ROM_Card"
         (path "/5ffe5182-cc98-4b6a-b75c-eae8ba1b784e"
-          (reference "SW2") (unit 1)
+          (reference "ID1") (unit 1)
         )
       )
@@
   (symbol (lib_id "Switch:SW_SPDT") (at 101.6 100.33 180) (unit 1)
     (in_bom yes) (on_board yes) (dnp no)
-    (property "Reference" "SW4" (at 100.33 100.33 0)
+    (property "Reference" "ID3" (at 100.33 100.33 0)
       (effects (font (size 1.27 1.27)))
     )
@@
       (project "ROM_Card"
         (path "/5ffe5182-cc98-4b6a-b75c-eae8ba1b784e"
-          (reference "SW4") (unit 1)
+          (reference "ID3") (unit 1)
         )
       )
@@
       (effects (font (size 1.27 1.27)) (justify left))
     )
-    (property "Footprint" "" (at 133.35 29.21 0)
+    (property "Footprint" "Package_SO:TSSOP-16_4.4x5mm_P0.65mm" (at 133.35 29.21 0)
       (effects (font (size 1.27 1.27)) hide)
     )
@@
   (symbol (lib_id "Switch:SW_SPDT") (at 183.515 66.04 180) (unit 1)
     (in_bom yes) (on_board yes) (dnp no)
-    (property "Reference" "SW10" (at 182.245 66.04 0)
+    (property "Reference" "SA14" (at 182.245 66.04 0)
       (effects (font (size 1.27 1.27)))
     )
@@
       (project "ROM_Card"
         (path "/5ffe5182-cc98-4b6a-b75c-eae8ba1b784e"
-          (reference "SW10") (unit 1)
+          (reference "SA14") (unit 1)
         )
       )
@@
   (symbol (lib_id "Switch:SW_SPDT") (at 101.6 92.71 180) (unit 1)
     (in_bom yes) (on_board yes) (dnp no)
-    (property "Reference" "SW3" (at 100.33 92.71 0)
+    (property "Reference" "ID2" (at 100.33 92.71 0)
       (effects (font (size 1.27 1.27)))
     )
@@
       (project "ROM_Card"
         (path "/5ffe5182-cc98-4b6a-b75c-eae8ba1b784e"
-          (reference "SW3") (unit 1)
+          (reference "ID2") (unit 1)
         )
       )
@@
   (symbol (lib_id "Switch:SW_SPDT") (at 101.6 123.19 180) (unit 1)
     (in_bom yes) (on_board yes) (dnp no)
-    (property "Reference" "SW7" (at 100.33 123.19 0)
+    (property "Reference" "ID6" (at 100.33 123.19 0)
       (effects (font (size 1.27 1.27)))
     )
@@
       (project "ROM_Card"
         (path "/5ffe5182-cc98-4b6a-b75c-eae8ba1b784e"
-          (reference "SW7") (unit 1)
+          (reference "ID6") (unit 1)
         )
       )
@@
   (symbol (lib_id "Switch:SW_SPDT") (at 101.6 107.95 180) (unit 1)
     (in_bom yes) (on_board yes) (dnp no)
-    (property "Reference" "SW5" (at 100.33 107.95 0)
+    (property "Reference" "ID4" (at 100.33 107.95 0)
       (effects (font (size 1.27 1.27)))
     )
@@
       (project "ROM_Card"
         (path "/5ffe5182-cc98-4b6a-b75c-eae8ba1b784e"
-          (reference "SW5") (unit 1)
-        )
-      )
+          (reference "ID4") (unit 1)
+        )
+      )
